File: KiCad/Open Interface III/USB_Isolated.kicad_sch (KiCad schematic)
At the start: 14 parts, among them J1 USB_B, U1 NUP4202, U2 ADUM4160

Commit message: OI III Schematics 0.1
Parts:
- C13: renamed from C1; footprint (none) -> Capacitor_SMD:C_1206_3216Metric_Pad1.33x1.80mm_HandSolder
- C14: renamed from C2; footprint (none) -> Capacitor_SMD:C_1206_3216Metric_Pad1.33x1.80mm_HandSolder
- C15: renamed from C3; footprint (none) -> Capacitor_SMD:C_1206_3216Metric_Pad1.33x1.80mm_HandSolder
- C16: renamed from C4; footprint (none) -> Capacitor_SMD:C_1206_3216Metric_Pad1.33x1.80mm_HandSolder
- J2: renamed from J1; footprint (none) -> MyFootprints:USB_B_OST_USB-B1HSxx_Horizontal
- L1, L2, L3, L4: footprint (none) -> Inductor_SMD:L_1206_3216Metric_Pad1.22x1.90mm_HandSolder
- R11: renamed from R1; footprint (none) -> Resistor_SMD:R_1206_3216Metric_Pad1.30x1.75mm_HandSolder
- R12: renamed from R2; footprint (none) -> Resistor_SMD:R_1206_3216Metric_Pad1.30x1.75mm_HandSolder
- R13: renamed from R3; footprint (none) -> Resistor_SMD:R_1206_3216Metric_Pad1.30x1.75mm_HandSolder
- renumbered U1 to U3, U2 to U4
Changed lines of the file:
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@@
 	(generator_version "8.0")
 	(paper "A4")
+	(title_block
+		(rev "0.1")
+	)
 	(junction
 		(at 109.22 132.08)
@@
 		(dnp no)
 		(fields_autoplaced yes)
-		(property "Reference" "R2"
+		(property "Reference" "R12"
 			(at 135.89 100.33 90)
 			(effects
@@
 			)
 		)
-		(property "Footprint" ""
+		(property "Footprint" "Resistor_SMD:R_1206_3216Metric_Pad1.30x1.75mm_HandSolder"
 			(at 135.89 108.458 90)
 			(effects
@@
 			(project ""
 				(path "/d93537ee-5c24-4c3e-8ba0-9c6559a17368/38dbc9f8-2c26-4fae-962d-1a1a74211f12"
-					(reference "R2")
+					(reference "R12")
 					(unit 1)
 				)
@@
 		(dnp no)
 		(fields_autoplaced yes)
-		(property "Reference" "#PWR2"
+		(property "Reference" "#PWR14"
 			(at 172.72 142.24 0)
 			(effects
@@
 			(project ""
 				(path "/d93537ee-5c24-4c3e-8ba0-9c6559a17368/38dbc9f8-2c26-4fae-962d-1a1a74211f12"
-					(reference "#PWR2")
+					(reference "#PWR14")
 					(unit 1)
 				)
@@
 		(dnp no)
 		(fields_autoplaced yes)
-		(property "Reference" "R3"
+		(property "Reference" "R13"
 			(at 135.89 110.49 90)
 			(effects
@@
 			)
 		)
-		(property "Footprint" ""
+		(property "Footprint" "Resistor_SMD:R_1206_3216Metric_Pad1.30x1.75mm_HandSolder"
 			(at 135.89 118.618 90)
 			(effects
@@
 			(project "Open Interface III"
 				(path "/d93537ee-5c24-4c3e-8ba0-9c6559a17368/38dbc9f8-2c26-4fae-962d-1a1a74211f12"
-					(reference "R3")
+					(reference "R13")
 					(unit 1)
 				)
@@
 			)
 		)
-		(property "Footprint" ""
+		(property "Footprint" "Inductor_SMD:L_1206_3216Metric_Pad1.22x1.90mm_HandSolder"
 			(at 123.19 106.68 0)
 			(effects
@@
 		(dnp no)
 		(fields_autoplaced yes)
-		(property "Reference" "#PWR3"
+		(property "Reference" "#PWR15"
 			(at 195.58 74.93 0)
 			(effects
@@
 			(project ""
 				(path "/d93537ee-5c24-4c3e-8ba0-9c6559a17368/38dbc9f8-2c26-4fae-962d-1a1a74211f12"
-					(reference "#PWR3")
+					(reference "#PWR15")
 					(unit 1)
 				)
@@
 		(dnp no)
 		(fields_autoplaced yes)
-		(property "Reference" "U2"
+		(property "Reference" "U4"
 			(at 172.3741 91.44 0)
 			(effects
@@
 			(project ""
 				(path "/d93537ee-5c24-4c3e-8ba0-9c6559a17368/38dbc9f8-2c26-4fae-962d-1a1a74211f12"
-					(reference "U2")
+					(reference "U4")
 					(unit 1)
 				)
@@
 		(dnp no)
 		(fields_autoplaced yes)
-		(property "Reference" "C1"
+		(property "Reference" "C13"
 			(at 153.67 69.8499 0)
 			(effects
@@
 			)
 		)
-		(property "Footprint" ""
+		(property "Footprint" "Capacitor_SMD:C_1206_3216Metric_Pad1.33x1.80mm_HandSolder"
 			(at 150.8252 74.93 0)
 			(effects
@@
 			(project "Open Interface III"
 				(path "/d93537ee-5c24-4c3e-8ba0-9c6559a17368/38dbc9f8-2c26-4fae-962d-1a1a74211f12"
-					(reference "C1")
+					(reference "C13")
 					(unit 1)
 				)
@@
 		(dnp no)
 		(fields_autoplaced yes)
-		(property "Reference" "C2"
+		(property "Reference" "C14"
 			(at 153.67 87.6299 0)
 			(effects
@@
 			)
 		)
-		(property "Footprint" ""
+		(property "Footprint" "Capacitor_SMD:C_1206_3216Metric_Pad1.33x1.80mm_HandSolder"
 			(at 150.8252 92.71 0)
 			(effects
@@
 			(project "Open Interface III"
 				(path "/d93537ee-5c24-4c3e-8ba0-9c6559a17368/38dbc9f8-2c26-4fae-962d-1a1a74211f12"
-					(reference "C2")
+					(reference "C14")
 					(unit 1)
 				)
@@
 		(dnp no)
 		(fields_autoplaced yes)
-		(property "Reference" "R1"
+		(property "Reference" "R11"
 			(at 111.76 62.2299 0)
 			(effects
@@
 			)
 		)
-		(property "Footprint" ""
+		(property "Footprint" "Resistor_SMD:R_1206_3216Metric_Pad1.30x1.75mm_HandSolder"
 			(at 107.442 63.5 90)
 			(effects
@@
 			(project ""
 				(path "/d93537ee-5c24-4c3e-8ba0-9c6559a17368/38dbc9f8-2c26-4fae-962d-1a1a74211f12"
-					(reference "R1")
+					(reference "R11")
 					(unit 1)
 				)
@@
 			)
 		)
-		(property "Footprint" ""
+		(property "Footprint" "Inductor_SMD:L_1206_3216Metric_Pad1.22x1.90mm_HandSolder"
 			(at 195.58 80.01 0)
 			(effects
@@
 		(dnp no)
 		(fields_autoplaced yes)
-		(property "Reference" "J1"
+		(property "Reference" "J2"
 			(at 77.47 93.98 0)
 			(effects
@@
 			)
 		)
-		(property "Footprint" ""
+		(property "Footprint" "MyFootprints:USB_B_OST_USB-B1HSxx_Horizontal"
 			(at 81.28 107.95 0)
 			(effects
@@
 			(project ""
 				(path "/d93537ee-5c24-4c3e-8ba0-9c6559a17368/38dbc9f8-2c26-4fae-962d-1a1a74211f12"
-					(reference "J1")
+					(reference "J2")
 					(unit 1)
 				)
@@
 		(dnp no)
 		(fields_autoplaced yes)
-		(property "Reference" "#PWR1"
+		(property "Reference" "#PWR13"
 			(at 74.93 142.24 0)
 			(effects
@@
 			(project ""
 				(path "/d93537ee-5c24-4c3e-8ba0-9c6559a17368/38dbc9f8-2c26-4fae-962d-1a1a74211f12"
-					(reference "#PWR1")
+					(reference "#PWR13")
 					(unit 1)
 				)
@@
 			)
 		)
-		(property "Footprint" ""
+		(property "Footprint" "Inductor_SMD:L_1206_3216Metric_Pad1.22x1.90mm_HandSolder"
 			(at 123.19 116.84 0)
 			(effects
@@
 		(dnp no)
 		(fields_autoplaced yes)
-		(property "Reference" "C4"
+		(property "Reference" "C16"
 			(at 199.39 120.6499 0)
 			(effects
@@
 			)
 		)
-		(property "Footprint" ""
+		(property "Footprint" "Capacitor_SMD:C_1206_3216Metric_Pad1.33x1.80mm_HandSolder"
 			(at 196.5452 125.73 0)
 			(effects
@@
 			(project ""
 				(path "/d93537ee-5c24-4c3e-8ba0-9c6559a17368/38dbc9f8-2c26-4fae-962d-1a1a74211f12"
-					(reference "C4")
+					(reference "C16")
 					(unit 1)
 				)
@@
 		(dnp no)
 		(fields_autoplaced yes)
-		(property "Reference" "C3"
+		(property "Reference" "C15"
 			(at 199.39 96.5199 0)
 			(effects
@@
 			)
 		)
-		(property "Footprint" ""
+		(property "Footprint" "Capacitor_SMD:C_1206_3216Metric_Pad1.33x1.80mm_HandSolder"
 			(at 196.5452 101.6 0)
 			(effects
@@
 			(project "Open Interface III"
 				(path "/d93537ee-5c24-4c3e-8ba0-9c6559a17368/38dbc9f8-2c26-4fae-962d-1a1a74211f12"
-					(reference "C3")
+					(reference "C15")
 					(unit 1)
 				)
@@
 		(dnp no)
 		(fields_autoplaced yes)
-		(property "Reference" "U1"
+		(property "Reference" "U3"
 			(at 115.57 78.7399 0)
 			(effects
@@
 			(project ""
 				(path "/d93537ee-5c24-4c3e-8ba0-9c6559a17368/38dbc9f8-2c26-4fae-962d-1a1a74211f12"
-					(reference "U1")
+					(reference "U3")
 					(unit 1)
 				)
@@
 			)
 		)
-		(property "Footprint" ""
+		(property "Footprint" "Inductor_SMD:L_1206_3216Metric_Pad1.22x1.90mm_HandSolder"
 			(at 90.17 63.5 0)
 			(effects
