File: KiCad/Open Interface III/ACC.kicad_sch (KiCad schematic)
At the start: 0 parts

Commit message: OI III Schematics 0.1
Parts:
- added J10: UART, symbol My_Headers:3-pin_UART_Header
- added J11: HDMI_A, symbol Connector:HDMI_A
Connections:
- new net +5V: J11.18 (+5V)
- new net A11: J11.19 (HPD)
- new net A3: J11.12 (CK-)
- new net A4: J11.13 (CEC)
- new net A8: J11.14 (UTILITY)
- new net A9: J11.17 (GND)
- new net D11: J11.9 (D0-)
- new net D12: J11.10 (CK+)
- new net D13: J11.5 (D1S)
- new net D30: J11.7 (D0+)
- new net D32: J11.8 (D0S)
- new net D38: J11.11 (CKS)
- new net D47: J11.4 (D1+)
- new net D5: J11.6 (D1-)
- new net GND: J10.3 (Pin_3), J11.2 (D2S), J11.SH
- new net RxD3: J10.1 (Pin_1), J11.1 (D2+)
- new net SCL: J11.15 (SCL)
- new net SDA: J11.16 (SDA)
- new net TxD3: J10.2 (Pin_2), J11.3 (D2-)

Commit message: PCB 0.1, BOM
Parts:
- J10: footprint (none) -> Connector_PinHeader_2.54mm:PinHeader_1x03_P2.54mm_Vertical
- J11: footprint (none) -> MyFootprints:HDMI_A_Kycon_KDMIX-SL1-NS-WS-B15_VerticalRightAngle
Changed lines of the file:
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@@
 			)
 		)
-		(property "Footprint" ""
+		(property "Footprint" "Connector_PinHeader_2.54mm:PinHeader_1x03_P2.54mm_Vertical"
 			(at 70.358 48.006 0)
 			(effects
@@
 			)
 		)
-		(property "Footprint" ""
+		(property "Footprint" "MyFootprints:HDMI_A_Kycon_KDMIX-SL1-NS-WS-B15_VerticalRightAngle"
 			(at 154.305 77.47 0)
 			(effects
