File: KiCad/Open Interface III/Audio_Switching.kicad_sch (KiCad schematic)
At the start: 0 parts

Commit message: OI III Schematics 0.1
Parts:
- added C83, C84, C85, C86: 4.7n, symbol Device:C
- added C87: 10u, symbol Device:C_Polarized
- added D35, D36: 1N4148, symbol Diode:1N4148
- added J9: Mic In, symbol Connector_Audio:AudioJack2_Dual_Ground_Switch
- added JP7: DC to Mic, symbol Jumper:Jumper_2_Bridged
- added K2, K3: G5V-1, symbol Relay:G5V-1
- added L28, L29, L30, L31: 10uH, symbol Device:L
- added Q5: BC817, symbol Transistor_BJT:BC817
- added Q6: BC856B, symbol Transistor_BJT:BC856
- added R83: 10k, symbol Device:R
- added R84, R85: 1k5, symbol Device:R
- added RV5: 10k, symbol Device:R_Potentiometer
- added U24, U25: 2 x RCA Jack, symbol My_Parts:Dual_RCA_Jack
Connections:
- new net: C87.1, J9.T1, JP7.2 (B)
- new net: D35.2 (A), K2.9, Q5.3 (C)
- new net: Q6.1 (B), R84.2
- new net: D36.2 (A), K3.9, Q6.2 (E)
- new net: L31.1, U24.2
- new net: L28.1, U24.3
- new net: C87.2, JP7.1 (A), K3.10
- new net: L30.2, U25.3
- new net: L29.2, U25.2
- new net: K2.1, RV5.3
- new net: K3.1, RV5.2
- new net: Q5.1 (B), R85.2
- new net +5V: D35.1 (K), D36.1 (K), K2.2, K3.2, R83.1
- new net AFSK: R85.1
- new net GND: C83.2, C84.2, C85.2, C86.2, Q5.2 (E), Q6.3 (C), U24.1, U25.1
- new net Interlock In: C84.1, L29.1
- new net Mic Out: K3.5, K3.6
- new net PA PTT Out: C85.1, L30.1
- new net PTT from Foot: C86.1, L31.2, R83.2, R84.1
- new net SEQ Out: C83.1, L28.2
- new net Tx Audio: K2.10
- new net Tx Audio GND: RV5.1
- new net Tx Sound: K2.5, K2.6
Other:
- note added: "Foot PTT"
- note added: "Interlock In"
- note added: "PA PTT"
- note added: "Sequencer"

Commit message: PCB 0.1, BOM
Parts:
- removed J9: Mic In, symbol Connector_Audio:AudioJack2_Dual_Ground_Switch
- added J9: Mic In, MyFootprints:3,5mm Jack Panel Socket 3-pole Switch large, symbol Connector_Audio:AudioJack2_Ground_Switch
- C83, C84, C85, C86: footprint (none) -> Capacitor_SMD:C_1206_3216Metric_Pad1.33x1.80mm_HandSolder
- C87: footprint (none) -> Capacitor_SMD:CP_Elec_5x5.4
- D35, D36: footprint (none) -> Diode_SMD:D_SOD-523
- JP7: footprint (none) -> Connector_PinHeader_2.54mm:PinHeader_1x02_P2.54mm_Vertical
- K2, K3: footprint (none) -> Relay_THT:Relay_SPDT_Omron_G5V-1
- L28, L29, L30, L31: footprint (none) -> Inductor_SMD:L_1206_3216Metric_Pad1.22x1.90mm_HandSolder
- Q5, Q6: footprint (none) -> Package_TO_SOT_SMD:SOT-23-3
- R83, R84, R85: footprint (none) -> Resistor_SMD:R_1206_3216Metric_Pad1.30x1.75mm_HandSolder
- RV5: footprint (none) -> MyFootprints:3-pin JST Potentiometer
- U24, U25: footprint (none) -> MyFootprints:pro-signal PSG01550 Dual 2× RCA Phono SocketRight Angle PCB
Connections:
- net Tx Audio GND: now also J9.G
- net at C87.1, JP7.2 (B): now also J9.T
