File: KiCad/Open Interface III/DC-DC_Power.kicad_sch (KiCad schematic)
At the start: 17 parts, among them J6 Barrel_Jack_Switch, U13 LM2576HVS-5, U14 L78L33_SOT89

Commit message: OI III Schematics 0.1
Parts:
- D6: renamed from D4; footprint Diode_SMD:D_SMC -> (none)
- D7: renamed from D5; footprint Diode_SMD:D_SMC -> (none)
- D8: renamed from D3; footprint Diode_SMD:D_SMC -> (none)
- U15: renamed from U13; footprint Package_TO_SOT_SMD:TO-263-5_TabPin3 -> (none)
- U16: renamed from U14; footprint Package_TO_SOT_SMD:SOT-89-3 -> (none)
- renumbered C25 to C36, C30 to C37, C26 to C38, C29 to C39, C27 to C40, C28 to C41, C31 to C42, C24 to C43, J6 to J7, L25 to L24, L24 to L25
Changed lines of the file:
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@@
 	(generator_version "8.0")
 	(paper "A4")
+	(title_block
+		(rev "0.1")
+	)
 	(junction
 		(at 181.61 110.49)
@@
 		(dnp no)
 		(fields_autoplaced yes)
-		(property "Reference" "U13"
+		(property "Reference" "U15"
 			(at 163.83 45.72 0)
 			(effects
@@
 			)
 		)
-		(property "Footprint" "Package_TO_SOT_SMD:TO-263-5_TabPin3"
+		(property "Footprint" ""
 			(at 163.83 62.23 0)
 			(effects
@@
 			(project ""
 				(path "/d93537ee-5c24-4c3e-8ba0-9c6559a17368/f51ea176-0284-463d-bcc7-8a64c07392ab"
-					(reference "U13")
+					(reference "U15")
 					(unit 1)
 				)
@@
 		(dnp no)
 		(fields_autoplaced yes)
-		(property "Reference" "L25"
+		(property "Reference" "L24"
 			(at 115.57 30.48 90)
 			(effects
@@
 			(project "Open Interface III"
 				(path "/d93537ee-5c24-4c3e-8ba0-9c6559a17368/f51ea176-0284-463d-bcc7-8a64c07392ab"
-					(reference "L25")
+					(reference "L24")
 					(unit 1)
 				)
@@
 		(dnp no)
 		(fields_autoplaced yes)
-		(property "Reference" "C26"
+		(property "Reference" "C38"
 			(at 135.89 66.0399 0)
 			(effects
@@
 			(project ""
 				(path "/d93537ee-5c24-4c3e-8ba0-9c6559a17368/f51ea176-0284-463d-bcc7-8a64c07392ab"
-					(reference "C26")
+					(reference "C38")
 					(unit 1)
 				)
@@
 		(dnp no)
 		(fields_autoplaced yes)
-		(property "Reference" "#PWR47"
+		(property "Reference" "#PWR58"
 			(at 163.83 142.24 0)
 			(effects
@@
 			(project "Open Interface III"
 				(path "/d93537ee-5c24-4c3e-8ba0-9c6559a17368/f51ea176-0284-463d-bcc7-8a64c07392ab"
-					(reference "#PWR47")
+					(reference "#PWR58")
 					(unit 1)
 				)
@@
 		(dnp no)
 		(fields_autoplaced yes)
-		(property "Reference" "C27"
+		(property "Reference" "C40"
 			(at 149.86 117.2209 0)
 			(effects
@@
 			(project "Open Interface III"
 				(path "/d93537ee-5c24-4c3e-8ba0-9c6559a17368/f51ea176-0284-463d-bcc7-8a64c07392ab"
-					(reference "C27")
+					(reference "C40")
 					(unit 1)
 				)
@@
 		(dnp no)
 		(fields_autoplaced yes)
-		(property "Reference" "C31"
+		(property "Reference" "C42"
 			(at 198.12 118.1099 0)
 			(effects
@@
 			(project "Open Interface III"
 				(path "/d93537ee-5c24-4c3e-8ba0-9c6559a17368/f51ea176-0284-463d-bcc7-8a64c07392ab"
-					(reference "C31")
+					(reference "C42")
 					(unit 1)
 				)
@@
 		(dnp no)
 		(fields_autoplaced yes)
-		(property "Reference" "J6"
+		(property "Reference" "J7"
 			(at 64.77 41.91 0)
 			(effects
@@
 			(project ""
 				(path "/d93537ee-5c24-4c3e-8ba0-9c6559a17368/f51ea176-0284-463d-bcc7-8a64c07392ab"
-					(reference "J6")
+					(reference "J7")
 					(unit 1)
 				)
@@
 		(dnp no)
 		(fields_autoplaced yes)
-		(property "Reference" "#PWR44"
+		(property "Reference" "#PWR60"
 			(at 203.2 45.72 0)
 			(effects
@@
 			(project ""
 				(path "/d93537ee-5c24-4c3e-8ba0-9c6559a17368/f51ea176-0284-463d-bcc7-8a64c07392ab"
-					(reference "#PWR44")
+					(reference "#PWR60")
 					(unit 1)
 				)
@@
 		(dnp no)
 		(fields_autoplaced yes)
-		(property "Reference" "C29"
+		(property "Reference" "C39"
 			(at 135.89 118.1099 0)
 			(effects
@@
 			(project "Open Interface III"
 				(path "/d93537ee-5c24-4c3e-8ba0-9c6559a17368/f51ea176-0284-463d-bcc7-8a64c07392ab"
-					(reference "C29")
+					(reference "C39")
 					(unit 1)
 				)
@@
 		(dnp no)
 		(fields_autoplaced yes)
-		(property "Reference" "D5"
+		(property "Reference" "D7"
 			(at 86.6775 41.91 0)
 			(effects
@@
 			)
 		)
-		(property "Footprint" "Diode_SMD:D_SMC"
+		(property "Footprint" ""
 			(at 85.852 39.116 0)
 			(effects
@@
 			(project "Open Interface III"
 				(path "/d93537ee-5c24-4c3e-8ba0-9c6559a17368/f51ea176-0284-463d-bcc7-8a64c07392ab"
-					(reference "D5")
+					(reference "D7")
 					(unit 1)
 				)
@@
 		(dnp no)
 		(fields_autoplaced yes)
-		(property "Reference" "C30"
+		(property "Reference" "C37"
 			(at 121.92 118.1099 0)
 			(effects
@@
 			(project "Open Interface III"
 				(path "/d93537ee-5c24-4c3e-8ba0-9c6559a17368/f51ea176-0284-463d-bcc7-8a64c07392ab"
-					(reference "C30")
+					(reference "C37")
 					(unit 1)
 				)
@@
 		(dnp no)
 		(fields_autoplaced yes)
-		(property "Reference" "L24"
+		(property "Reference" "L25"
 			(at 193.04 53.34 90)
 			(effects
@@
 			(project ""
 				(path "/d93537ee-5c24-4c3e-8ba0-9c6559a17368/f51ea176-0284-463d-bcc7-8a64c07392ab"
-					(reference "L24")
+					(reference "L25")
 					(unit 1)
 				)
@@
 		(dnp no)
 		(fields_autoplaced yes)
-		(property "Reference" "C28"
+		(property "Reference" "C41"
 			(at 185.42 117.2209 0)
 			(effects
@@
 			(project "Open Interface III"
 				(path "/d93537ee-5c24-4c3e-8ba0-9c6559a17368/f51ea176-0284-463d-bcc7-8a64c07392ab"
-					(reference "C28")
+					(reference "C41")
 					(unit 1)
 				)
@@
 		(dnp no)
 		(fields_autoplaced yes)
-		(property "Reference" "#PWR43"
+		(property "Reference" "#PWR57"
 			(at 163.83 87.63 0)
 			(effects
@@
 			(project ""
 				(path "/d93537ee-5c24-4c3e-8ba0-9c6559a17368/f51ea176-0284-463d-bcc7-8a64c07392ab"
-					(reference "#PWR43")
+					(reference "#PWR57")
 					(unit 1)
 				)
@@
 		(dnp no)
 		(fields_autoplaced yes)
-		(property "Reference" "#PWR45"
+		(property "Reference" "#PWR56"
 			(at 118.11 105.41 0)
 			(effects
@@
 			(project "Open Interface III"
 				(path "/d93537ee-5c24-4c3e-8ba0-9c6559a17368/f51ea176-0284-463d-bcc7-8a64c07392ab"
-					(reference "#PWR45")
+					(reference "#PWR56")
 					(unit 1)
 				)
@@
 		(dnp no)
 		(fields_autoplaced yes)
-		(property "Reference" "C25"
+		(property "Reference" "C36"
 			(at 119.38 65.1509 0)
 			(effects
@@
 			(project "Open Interface III"
 				(path "/d93537ee-5c24-4c3e-8ba0-9c6559a17368/f51ea176-0284-463d-bcc7-8a64c07392ab"
-					(reference "C25")
+					(reference "C36")
 					(unit 1)
 				)
@@
 		(dnp no)
 		(fields_autoplaced yes)
-		(property "Reference" "C24"
+		(property "Reference" "C43"
 			(at 207.01 65.1509 0)
 			(effects
@@
 			(project ""
 				(path "/d93537ee-5c24-4c3e-8ba0-9c6559a17368/f51ea176-0284-463d-bcc7-8a64c07392ab"
-					(reference "C24")
+					(reference "C43")
 					(unit 1)
 				)
@@
 		(dnp no)
 		(fields_autoplaced yes)
-		(property "Reference" "D3"
+		(property "Reference" "D8"
 			(at 184.15 65.7224 90)
 			(effects
@@
 			)
 		)
-		(property "Footprint" "Diode_SMD:D_SMC"
+		(property "Footprint" ""
 			(at 172.466 67.818 0)
 			(effects
@@
 			(project ""
 				(path "/d93537ee-5c24-4c3e-8ba0-9c6559a17368/f51ea176-0284-463d-bcc7-8a64c07392ab"
-					(reference "D3")
+					(reference "D8")
 					(unit 1)
 				)
@@
 		(dnp no)
 		(fields_autoplaced yes)
-		(property "Reference" "U14"
+		(property "Reference" "U16"
 			(at 163.83 104.14 0)
 			(effects
@@
 			)
 		)
-		(property "Footprint" "Package_TO_SOT_SMD:SOT-89-3"
+		(property "Footprint" ""
 			(at 163.83 105.41 0)
 			(effects
@@
 			(project ""
 				(path "/d93537ee-5c24-4c3e-8ba0-9c6559a17368/f51ea176-0284-463d-bcc7-8a64c07392ab"
-					(reference "U14")
+					(reference "U16")
 					(unit 1)
 				)
@@
 		(dnp no)
 		(fields_autoplaced yes)
-		(property "Reference" "#PWR46"
+		(property "Reference" "#PWR59"
 			(at 194.31 105.41 0)
 			(effects
@@
 			(project ""
 				(path "/d93537ee-5c24-4c3e-8ba0-9c6559a17368/f51ea176-0284-463d-bcc7-8a64c07392ab"
-					(reference "#PWR46")
+					(reference "#PWR59")
 					(unit 1)
 				)
@@
 		(dnp no)
 		(fields_autoplaced yes)
-		(property "Reference" "D4"
+		(property "Reference" "D6"
 			(at 86.6775 29.21 0)
 			(effects
@@
 			)
 		)
-		(property "Footprint" "Diode_SMD:D_SMC"
+		(property "Footprint" ""
 			(at 85.852 26.416 0)
 			(effects
@@
 			(project "Open Interface III"
 				(path "/d93537ee-5c24-4c3e-8ba0-9c6559a17368/f51ea176-0284-463d-bcc7-8a64c07392ab"
-					(reference "D4")
+					(reference "D6")
 					(unit 1)
 				)

Commit message: PCB 0.1, BOM
Parts:
- C36: footprint (none) -> Capacitor_SMD:CP_Elec_8x10
- C37, C38, C39, C42: footprint (none) -> Capacitor_SMD:C_1206_3216Metric_Pad1.33x1.80mm_HandSolder
- C40, C41: footprint (none) -> Capacitor_SMD:CP_Elec_5x5.4
- C43: footprint (none) -> Capacitor_SMD:CP_Elec_8x10.5
- D6, D7, D8: footprint (none) -> Diode_SMD:D_SMB
- J7: footprint (none) -> MyFootprints:BarrelJack_Horizontal
- L24, L25: footprint (none) -> Inductor_SMD:L_1206_3216Metric_Pad1.22x1.90mm_HandSolder
- RV3: footprint (none) -> Varistor:RV_Disc_D12mm_W3.9mm_P7.5mm
- U15: footprint (none) -> Package_TO_SOT_SMD:TO-263-5_TabPin3
- U16: footprint (none) -> Package_TO_SOT_SMD:SOT-89-3_Handsoldering
Changed lines of the file:
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@@
 			)
 		)
-		(property "Footprint" ""
+		(property "Footprint" "Package_TO_SOT_SMD:TO-263-5_TabPin3"
 			(at 163.83 62.23 0)
 			(effects
@@
 			)
 		)
-		(property "Footprint" ""
+		(property "Footprint" "Inductor_SMD:L_1206_3216Metric_Pad1.22x1.90mm_HandSolder"
 			(at 115.57 35.56 0)
 			(effects
@@
 			)
 		)
-		(property "Footprint" ""
+		(property "Footprint" "Capacitor_SMD:C_1206_3216Metric_Pad1.33x1.80mm_HandSolder"
 			(at 133.0452 71.12 0)
 			(effects
@@
 			)
 		)
-		(property "Footprint" ""
+		(property "Footprint" "Varistor:RV_Disc_D12mm_W3.9mm_P7.5mm"
 			(at 97.282 67.31 90)
 			(effects
@@
 			)
 		)
-		(property "Footprint" ""
+		(property "Footprint" "Capacitor_SMD:CP_Elec_5x5.4"
 			(at 147.0152 123.19 0)
 			(effects
@@
 			)
 		)
-		(property "Footprint" ""
+		(property "Footprint" "Capacitor_SMD:C_1206_3216Metric_Pad1.33x1.80mm_HandSolder"
 			(at 195.2752 123.19 0)
 			(effects
@@
 			)
 		)
-		(property "Footprint" ""
+		(property "Footprint" "MyFootprints:BarrelJack_Horizontal"
 			(at 66.04 51.816 0)
 			(effects
@@
 			)
 		)
-		(property "Footprint" ""
+		(property "Footprint" "Capacitor_SMD:C_1206_3216Metric_Pad1.33x1.80mm_HandSolder"
 			(at 133.0452 123.19 0)
 			(effects
@@
 			)
 		)
-		(property "Footprint" ""
+		(property "Footprint" "Diode_SMD:D_SMB"
 			(at 85.852 39.116 0)
 			(effects
@@
 			)
 		)
-		(property "Footprint" ""
+		(property "Footprint" "Capacitor_SMD:C_1206_3216Metric_Pad1.33x1.80mm_HandSolder"
 			(at 119.0752 123.19 0)
 			(effects
@@
 			)
 		)
-		(property "Footprint" ""
+		(property "Footprint" "Inductor_SMD:L_1206_3216Metric_Pad1.22x1.90mm_HandSolder"
 			(at 193.04 58.42 0)
 			(effects
@@
 			)
 		)
-		(property "Footprint" ""
+		(property "Footprint" "Capacitor_SMD:CP_Elec_5x5.4"
 			(at 182.5752 123.19 0)
 			(effects
@@
 			)
 		)
-		(property "Footprint" ""
+		(property "Footprint" "Capacitor_SMD:CP_Elec_8x10"
 			(at 116.5352 71.12 0)
 			(effects
@@
 			)
 		)
-		(property "Footprint" ""
+		(property "Footprint" "Capacitor_SMD:CP_Elec_8x10.5"
 			(at 204.1652 71.12 0)
 			(effects
@@
 			)
 		)
-		(property "Footprint" ""
+		(property "Footprint" "Diode_SMD:D_SMB"
 			(at 172.466 67.818 0)
 			(effects
@@
 			)
 		)
-		(property "Footprint" ""
+		(property "Footprint" "Package_TO_SOT_SMD:SOT-89-3_Handsoldering"
 			(at 163.83 105.41 0)
 			(effects
@@
 			)
 		)
-		(property "Footprint" ""
+		(property "Footprint" "Diode_SMD:D_SMB"
 			(at 85.852 26.416 0)
 			(effects
