File: KiCad/Open Interface III/Micro_SD.kicad_sch (KiCad schematic)
At the start: 6 parts, among them J5 Micro_SD_Card_Det2, U11 LSF0102, U12 LSF0102

Commit message: OI III Schematics 0.1
Parts:
- U13: renamed from U11; footprint Package_TO_SOT_SMD:SOT-23-8 -> (none)
- U14: renamed from U12; footprint Package_TO_SOT_SMD:SOT-23-8 -> (none)
- renumbered C23 to C34, C22 to C35, J5 to J6, R42 to R52
Changed lines of the file:
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@@
 	(generator_version "8.0")
 	(paper "A4")
+	(title_block
+		(rev "0.1")
+	)
 	(junction
 		(at 143.51 80.01)
@@
 		(dnp no)
 		(fields_autoplaced yes)
-		(property "Reference" "#PWR39"
+		(property "Reference" "#PWR54"
 			(at 154.94 64.77 0)
 			(effects
@@
 			(project "Open Interface III"
 				(path "/d93537ee-5c24-4c3e-8ba0-9c6559a17368/604b6e8f-bbfc-4153-991d-cc7d34f8db00"
-					(reference "#PWR39")
+					(reference "#PWR54")
 					(unit 1)
 				)
@@
 		(dnp no)
 		(fields_autoplaced yes)
-		(property "Reference" "R42"
+		(property "Reference" "R52"
 			(at 71.12 59.6899 0)
 			(effects
@@
 			(project "Open Interface III"
 				(path "/d93537ee-5c24-4c3e-8ba0-9c6559a17368/604b6e8f-bbfc-4153-991d-cc7d34f8db00"
-					(reference "R42")
+					(reference "R52")
 					(unit 1)
 				)
@@
 		(dnp no)
 		(fields_autoplaced yes)
-		(property "Reference" "U11"
+		(property "Reference" "U13"
 			(at 130.81 62.23 0)
 			(effects
@@
 			)
 		)
-		(property "Footprint" "Package_TO_SOT_SMD:SOT-23-8"
+		(property "Footprint" ""
 			(at 134.62 99.822 0)
 			(effects
@@
 			(project "Open Interface III"
 				(path "/d93537ee-5c24-4c3e-8ba0-9c6559a17368/604b6e8f-bbfc-4153-991d-cc7d34f8db00"
-					(reference "U11")
+					(reference "U13")
 					(unit 1)
 				)
@@
 		(dnp no)
 		(fields_autoplaced yes)
-		(property "Reference" "U12"
+		(property "Reference" "U14"
 			(at 130.81 104.14 0)
 			(effects
@@
 			)
 		)
-		(property "Footprint" "Package_TO_SOT_SMD:SOT-23-8"
+		(property "Footprint" ""
 			(at 134.62 141.732 0)
 			(effects
@@
 			(project "Open Interface III"
 				(path "/d93537ee-5c24-4c3e-8ba0-9c6559a17368/604b6e8f-bbfc-4153-991d-cc7d34f8db00"
-					(reference "U12")
+					(reference "U14")
 					(unit 1)
 				)
@@
 		(dnp no)
 		(fields_autoplaced yes)
-		(property "Reference" "C22"
+		(property "Reference" "C35"
 			(at 158.75 119.3799 0)
 			(effects
@@
 			(project "Open Interface III"
 				(path "/d93537ee-5c24-4c3e-8ba0-9c6559a17368/604b6e8f-bbfc-4153-991d-cc7d34f8db00"
-					(reference "C22")
+					(reference "C35")
 					(unit 1)
 				)
@@
 		(dnp no)
 		(fields_autoplaced yes)
-		(property "Reference" "#PWR40"
+		(property "Reference" "#PWR55"
 			(at 154.94 144.78 0)
 			(effects
@@
 			(project "Open Interface III"
 				(path "/d93537ee-5c24-4c3e-8ba0-9c6559a17368/604b6e8f-bbfc-4153-991d-cc7d34f8db00"
-					(reference "#PWR40")
+					(reference "#PWR55")
 					(unit 1)
 				)
@@
 		(dnp no)
 		(fields_autoplaced yes)
-		(property "Reference" "J5"
+		(property "Reference" "J6"
 			(at 201.295 66.04 0)
 			(effects
@@
 			(project "Open Interface III"
 				(path "/d93537ee-5c24-4c3e-8ba0-9c6559a17368/604b6e8f-bbfc-4153-991d-cc7d34f8db00"
-					(reference "J5")
+					(reference "J6")
 					(unit 1)
 				)
@@
 		(dnp no)
 		(fields_autoplaced yes)
-		(property "Reference" "C23"
+		(property "Reference" "C34"
 			(at 72.39 129.5399 0)
 			(effects
@@
 			(project "Open Interface III"
 				(path "/d93537ee-5c24-4c3e-8ba0-9c6559a17368/604b6e8f-bbfc-4153-991d-cc7d34f8db00"
-					(reference "C23")
+					(reference "C34")
 					(unit 1)
 				)
@@
 		(dnp no)
 		(fields_autoplaced yes)
-		(property "Reference" "#PWR42"
+		(property "Reference" "#PWR52"
 			(at 68.58 55.88 0)
 			(effects
@@
 			(project "Open Interface III"
 				(path "/d93537ee-5c24-4c3e-8ba0-9c6559a17368/604b6e8f-bbfc-4153-991d-cc7d34f8db00"
-					(reference "#PWR42")
+					(reference "#PWR52")
 					(unit 1)
 				)
@@
 		(dnp no)
 		(fields_autoplaced yes)
-		(property "Reference" "#PWR41"
+		(property "Reference" "#PWR53"
 			(at 80.01 149.86 0)
 			(effects
@@
 			(project "Open Interface III"
 				(path "/d93537ee-5c24-4c3e-8ba0-9c6559a17368/604b6e8f-bbfc-4153-991d-cc7d34f8db00"
-					(reference "#PWR41")
+					(reference "#PWR53")
 					(unit 1)
 				)

Commit message: PCB 0.1, BOM
Parts:
- C34, C35: footprint (none) -> Capacitor_SMD:C_1206_3216Metric_Pad1.33x1.80mm_HandSolder
- J6: footprint (none) -> Connector_Card:microSD_HC_Hirose_DM3AT-SF-PEJM5
- R52: footprint (none) -> Resistor_SMD:R_1206_3216Metric_Pad1.30x1.75mm_HandSolder
- U13, U14: footprint (none) -> Package_TO_SOT_SMD:SOT-23W_Handsoldering
Changed lines of the file:
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@@
 			)
 		)
-		(property "Footprint" ""
+		(property "Footprint" "Resistor_SMD:R_1206_3216Metric_Pad1.30x1.75mm_HandSolder"
 			(at 70.358 60.96 90)
 			(effects
@@
 			)
 		)
-		(property "Footprint" ""
+		(property "Footprint" "Package_TO_SOT_SMD:SOT-23W_Handsoldering"
 			(at 134.62 99.822 0)
 			(effects
@@
 			)
 		)
-		(property "Footprint" ""
+		(property "Footprint" "Package_TO_SOT_SMD:SOT-23W_Handsoldering"
 			(at 134.62 141.732 0)
 			(effects
@@
 			)
 		)
-		(property "Footprint" ""
+		(property "Footprint" "Capacitor_SMD:C_1206_3216Metric_Pad1.33x1.80mm_HandSolder"
 			(at 155.9052 124.46 0)
 			(effects
@@
 			)
 		)
-		(property "Footprint" ""
+		(property "Footprint" "Connector_Card:microSD_HC_Hirose_DM3AT-SF-PEJM5"
 			(at 252.73 69.85 0)
 			(effects
@@
 			)
 		)
-		(property "Footprint" ""
+		(property "Footprint" "Capacitor_SMD:C_1206_3216Metric_Pad1.33x1.80mm_HandSolder"
 			(at 69.5452 134.62 0)
 			(effects
