File: KiCad/Open Interface III/Misc.kicad_sch (KiCad schematic)
At the start: 32 parts, among them J4 Paddle In, SW1 RotaryEncoder, U10 Mode, U5 USR-ES1 W5500, U6 LCD_HD44780, U7 Set, U8 M1, U9 M2

Commit message: OI III Schematics 0.1
Parts:
- U7: renamed from U6; footprint My_Parts:LCD_HD44780_16x2_w_headers_large -> (none)
- U8: renamed from U5; footprint MyFootprints:USR-ES1 W5500 -> (none)
- renumbered C13 to C25, C17 to C26, C20 to C27, C21 to C28, C18 to C29, C19 to C30, J4 to J3, JP3 to JP4, L22 to L6, L23 to L7, R23 to R33, R24 to R34, R25 to R35, R34 to R38, R32 to R39, R38 to R40, R39 to R41, R40 to R42, R33 to R43, R41 to R44, R35 to R45, U8 to U10, U9 to U11, U10 to U12, U7 to U9
Connections:
- net Enc-A renamed Enc A
- net Enc-B renamed Enc B
- net LCD-D4 renamed LCD D4
- net LCD-D5 renamed LCD D5
- net LCD-D6 renamed LCD D6
- net LCD-D8 renamed LCD D8
- net LCD-E renamed LCD E
- net LCD-RS renamed LCD RS

Commit message: PCB 0.1, BOM
Parts:
- removed J3: Paddle In, symbol Connector_Audio:AudioJack2_Dual_Ground_Switch
- added J3: Paddle In, MyFootprints:3,5mm Jack Panel Socket 3-pole Switch large, symbol Connector_Audio:AudioJack2_Ground_Switch
- C25, C26, C27, C28, C29, C30: footprint (none) -> Capacitor_SMD:C_1206_3216Metric_Pad1.33x1.80mm_HandSolder
- JP4: footprint (none) -> Connector_PinHeader_2.54mm:PinHeader_1x02_P2.54mm_Vertical
- L6, L7: footprint (none) -> Inductor_SMD:L_1206_3216Metric_Pad1.22x1.90mm_HandSolder
- R33, R34, R35, R36, R37, R38, R39, R40, R41, R42, R43, R44, R45: footprint (none) -> Resistor_SMD:R_1206_3216Metric_Pad1.30x1.75mm_HandSolder
- RV1, RV2: footprint (none) -> MyFootprints:3-pin JST Potentiometer
- SW1: footprint (none) -> MyFootprints:3-pin JST Rotary Encoder
- U10, U11, U12, U9: footprint (none) -> MyFootprints:2-pin JST Switch
- U7: footprint (none) -> MyFootprints:2 x 6-pin JST LCD HD44780 Stacked
- U8: footprint (none) -> MyFootprints:USR-ES1 W5500
Connections:
- net GND: now also J3.G
- net at L7.2: now also J3.S
- net at L6.2: now also J3.T
Changed lines of the file:
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@@
 			)
 		)
-		(property "Footprint" ""
+		(property "Footprint" "MyFootprints:3-pin JST Potentiometer"
 			(at 35.56 154.94 0)
 			(effects
@@
 			)
 		)
-		(property "Footprint" ""
+		(property "Footprint" "Resistor_SMD:R_1206_3216Metric_Pad1.30x1.75mm_HandSolder"
 			(at 225.552 140.97 90)
 			(effects
@@
 			)
 		)
-		(property "Footprint" ""
+		(property "Footprint" "Resistor_SMD:R_1206_3216Metric_Pad1.30x1.75mm_HandSolder"
 			(at 243.84 50.038 90)
 			(effects
@@
 			)
 		)
-		(property "Footprint" ""
+		(property "Footprint" "Resistor_SMD:R_1206_3216Metric_Pad1.30x1.75mm_HandSolder"
 			(at 193.802 118.11 90)
 			(effects
@@
 			)
 		)
-		(property "Footprint" ""
+		(property "Footprint" "Connector_PinHeader_2.54mm:PinHeader_1x02_P2.54mm_Vertical"
 			(at 52.07 175.26 0)
 			(effects
@@
 			)
 		)
-		(property "Footprint" ""
+		(property "Footprint" "Resistor_SMD:R_1206_3216Metric_Pad1.30x1.75mm_HandSolder"
 			(at 39.37 46.228 90)
 			(effects
@@
 			)
 		)
-		(property "Footprint" ""
+		(property "Footprint" "Capacitor_SMD:C_1206_3216Metric_Pad1.33x1.80mm_HandSolder"
 			(at 196.5452 144.78 0)
 			(effects
@@
 			)
 		)
-		(property "Footprint" ""
+		(property "Footprint" "MyFootprints:2 x 6-pin JST LCD HD44780 Stacked"
 			(at 66.04 87.63 0)
 			(effects
@@
 			)
 		)
-		(property "Footprint" ""
+		(property "Footprint" "Resistor_SMD:R_1206_3216Metric_Pad1.30x1.75mm_HandSolder"
 			(at 217.932 39.37 90)
 			(effects
@@
 			)
 		)
-		(property "Footprint" ""
+		(property "Footprint" "MyFootprints:2-pin JST Switch"
 			(at 236.22 153.67 0)
 			(effects
@@
 	)
 	(symbol
-		(lib_id "Connector_Audio:AudioJack2_Dual_Ground_Switch")
-		(at 149.86 114.3 0)
-		(unit 1)
-		(exclude_from_sim no)
-		(in_bom yes)
-		(on_board yes)
-		(dnp no)
-		(fields_autoplaced yes)
-		(property "Reference" "J3"
-			(at 148.5265 102.87 0)
-			(effects
-				(font
-					(size 1.27 1.27)
-				)
-			)
-		)
-		(property "Value" "Paddle In"
-			(at 148.5265 105.41 0)
-			(effects
-				(font
-					(size 1.27 1.27)
-				)
-			)
-		)
-		(property "Footprint" ""
-			(at 148.59 109.22 0)
-			(effects
-				(font
-					(size 1.27 1.27)
-				)
-				(hide yes)
-			)
-		)
-		(property "Datasheet" "~"
-			(at 148.59 109.22 0)
-			(effects
-				(font
-					(size 1.27 1.27)
-				)
-				(hide yes)
-			)
-		)
-		(property "Description" "Audio Jack, Dual, 2 Poles (Mono / TS), Grounded Sleeve, Switched Pole (Normalling)"
-			(at 149.86 114.3 0)
-			(effects
-				(font
-					(size 1.27 1.27)
-				)
-				(hide yes)
-			)
-		)
-		(pin "TN1"
-		)
-		(pin "SN1"
-		)
-		(pin "T2"
-		)
-		(pin "SN2"
-		)
-		(pin "TN2"
-		)
-		(pin "S2"
-		)
-		(pin "T1"
-		)
-		(pin "G"
-		)
-		(pin "S1"
-		)
-		(instances
-			(project "Open Interface III"
-				(path "/d93537ee-5c24-4c3e-8ba0-9c6559a17368/671112d9-5af4-4042-bb4b-eae8a0524e41"
-					(reference "J3")
-					(unit 1)
-				)
-			)
-		)
-	)
-	(symbol
 		(lib_id "Device:R_Potentiometer")
 		(at 90.17 137.16 90)
@@
 			)
 		)
-		(property "Footprint" ""
+		(property "Footprint" "MyFootprints:3-pin JST Potentiometer"
 			(at 90.17 137.16 0)
 			(effects
@@
 			)
 		)
-		(property "Footprint" ""
+		(property "Footprint" "Resistor_SMD:R_1206_3216Metric_Pad1.30x1.75mm_HandSolder"
 			(at 23.622 53.34 90)
 			(effects
@@
 			)
 		)
-		(property "Footprint" ""
+		(property "Footprint" "Inductor_SMD:L_1206_3216Metric_Pad1.22x1.90mm_HandSolder"
 			(at 186.69 118.11 0)
 			(effects
@@
 			)
 		)
-		(property "Footprint" ""
+		(property "Footprint" "Capacitor_SMD:C_1206_3216Metric_Pad1.33x1.80mm_HandSolder"
 			(at 174.9552 144.78 0)
 			(effects
@@
 			)
 		)
-		(property "Footprint" ""
+		(property "Footprint" "Capacitor_SMD:C_1206_3216Metric_Pad1.33x1.80mm_HandSolder"
 			(at 202.8952 66.04 0)
 			(effects
@@
 			)
 		)
-		(property "Footprint" ""
+		(property "Footprint" "Capacitor_SMD:C_1206_3216Metric_Pad1.33x1.80mm_HandSolder"
 			(at 54.3052 57.15 0)
 			(effects
@@
 			)
 		)
-		(property "Footprint" ""
+		(property "Footprint" "MyFootprints:3-pin JST Rotary Encoder"
 			(at 223.266 67.31 0)
 			(effects
@@
 			)
 		)
-		(property "Footprint" ""
+		(property "Footprint" "Resistor_SMD:R_1206_3216Metric_Pad1.30x1.75mm_HandSolder"
 			(at 242.57 100.838 90)
 			(effects
@@
 			)
 		)
-		(property "Footprint" ""
+		(property "Footprint" "Resistor_SMD:R_1206_3216Metric_Pad1.30x1.75mm_HandSolder"
 			(at 210.82 50.038 90)
 			(effects
@@
 			)
 		)
-		(property "Footprint" ""
+		(property "Footprint" "Resistor_SMD:R_1206_3216Metric_Pad1.30x1.75mm_HandSolder"
 			(at 233.172 39.37 90)
 			(effects
@@
 			)
 		)
-		(property "Footprint" ""
+		(property "Footprint" "Resistor_SMD:R_1206_3216Metric_Pad1.30x1.75mm_HandSolder"
 			(at 229.108 105.41 90)
 			(effects
@@
 			)
 		)
-		(property "Footprint" ""
+		(property "Footprint" "MyFootprints:2-pin JST Switch"
 			(at 259.08 105.41 0)
 			(effects
@@
 			)
 		)
-		(property "Footprint" ""
+		(property "Footprint" "Resistor_SMD:R_1206_3216Metric_Pad1.30x1.75mm_HandSolder"
 			(at 225.552 123.19 90)
 			(effects
@@
 			)
 		)
-		(property "Footprint" ""
+		(property "Footprint" "Resistor_SMD:R_1206_3216Metric_Pad1.30x1.75mm_HandSolder"
 			(at 23.622 35.56 90)
 			(effects
@@
 			)
 		)
-		(property "Footprint" ""
+		(property "Footprint" "MyFootprints:USR-ES1 W5500"
 			(at 151.13 58.42 0)
 			(effects
@@
 	)
 	(symbol
+		(lib_id "Connector_Audio:AudioJack2_Ground_Switch")
+		(at 149.86 114.3 0)
+		(unit 1)
+		(exclude_from_sim no)
+		(in_bom yes)
+		(on_board yes)
+		(dnp no)
+		(fields_autoplaced yes)
+		(property "Reference" "J3"
+			(at 149.225 102.87 0)
+			(effects
+				(font
+					(size 1.27 1.27)
+				)
+			)
+		)
+		(property "Value" "Paddle In"
+			(at 149.225 105.41 0)
+			(effects
+				(font
+					(size 1.27 1.27)
+				)
+			)
+		)
+		(property "Footprint" "MyFootprints:3,5mm Jack Panel Socket 3-pole Switch large"
+			(at 149.86 109.22 0)
+			(effects
+				(font
+					(size 1.27 1.27)
+				)
+				(hide yes)
+			)
+		)
+		(property "Datasheet" "~"
+			(at 149.86 109.22 0)
+			(effects
+				(font
+					(size 1.27 1.27)
+				)
+				(hide yes)
+			)
+		)
+		(property "Description" "Audio Jack, 2 Poles (Mono / TS), Grounded Sleeve, Switched Pole (Normalling)"
+			(at 149.86 114.3 0)
+			(effects
+				(font
+					(size 1.27 1.27)
+				)
+				(hide yes)
+			)
+		)
+		(pin "TN"
+		)
+		(pin "G"
+		)
+		(pin "S"
+		)
+		(pin "SN"
+		)
+		(pin "T"
+		)
+		(instances
+			(project ""
+				(path "/d93537ee-5c24-4c3e-8ba0-9c6559a17368/671112d9-5af4-4042-bb4b-eae8a0524e41"
+					(reference "J3")
+					(unit 1)
+				)
+			)
+		)
+	)
+	(symbol
 		(lib_id "Device:C")
 		(at 161.29 62.23 0)
@@
 			)
 		)
-		(property "Footprint" ""
+		(property "Footprint" "Capacitor_SMD:C_1206_3216Metric_Pad1.33x1.80mm_HandSolder"
 			(at 162.2552 66.04 0)
 			(effects
@@
 			)
 		)
-		(property "Footprint" ""
+		(property "Footprint" "Inductor_SMD:L_1206_3216Metric_Pad1.22x1.90mm_HandSolder"
 			(at 165.1 123.19 0)
 			(effects
@@
 			)
 		)
-		(property "Footprint" ""
+		(property "Footprint" "MyFootprints:2-pin JST Switch"
 			(at 236.22 135.89 0)
 			(effects
@@
 			)
 		)
-		(property "Footprint" ""
+		(property "Footprint" "Resistor_SMD:R_1206_3216Metric_Pad1.30x1.75mm_HandSolder"
 			(at 172.212 123.19 90)
 			(effects
@@
 			)
 		)
-		(property "Footprint" ""
+		(property "Footprint" "MyFootprints:2-pin JST Switch"
 			(at 236.22 118.11 0)
 			(effects
@@
 			)
 		)
-		(property "Footprint" ""
+		(property "Footprint" "Capacitor_SMD:C_1206_3216Metric_Pad1.33x1.80mm_HandSolder"
 			(at 253.6952 66.04 0)
 			(effects
