File: KiCad/Open Interface III/Open Interface III.kicad_pcb (KiCad board)
At the start: 2 copper layers, 14 parts, among them J2 USB_B, U3 NUP4202, U4 ADUM4160

Commit message: PCB 0.1, BOM
Parts:
- added C1: 22p, Capacitor_SMD:C_1206_3216Metric_Pad1.33x1.80mm_HandSolder, F.Cu at (171.1, 85.1)
- added C10: 100n, Capacitor_SMD:C_1206_3216Metric_Pad1.33x1.80mm_HandSolder, F.Cu at (147.0, 76.2)
- added C11: 100n, Capacitor_SMD:C_1206_3216Metric_Pad1.33x1.80mm_HandSolder, F.Cu at (150.8, 76.2)
- added C12: 100n, Capacitor_SMD:C_1206_3216Metric_Pad1.33x1.80mm_HandSolder, F.Cu at (154.6, 76.2)
- added C17: 22p, Capacitor_SMD:C_1206_3216Metric_Pad1.33x1.80mm_HandSolder, F.Cu at (88.5, 87.4)
- added C18: 22p, Capacitor_SMD:C_1206_3216Metric_Pad1.33x1.80mm_HandSolder, F.Cu at (82.8, 92.5)
- added C19: 27p, Capacitor_SMD:C_1206_3216Metric_Pad1.33x1.80mm_HandSolder, F.Cu at (70.1, 86.8)
- added C2: 4.7n, Capacitor_SMD:C_1206_3216Metric_Pad1.33x1.80mm_HandSolder, F.Cu at (187.6, 86.7)
- added C20: 27p, Capacitor_SMD:C_1206_3216Metric_Pad1.33x1.80mm_HandSolder, F.Cu at (70.1, 75.4)
- added C21: 4.7u, Capacitor_SMD:CP_Elec_4x5.4, F.Cu at (160.4, 109.6)
- added C22: 22p, Capacitor_SMD:C_1206_3216Metric_Pad1.33x1.80mm_HandSolder, F.Cu at (173.1, 116.1)
- added C23: 22p, Capacitor_SMD:C_1206_3216Metric_Pad1.33x1.80mm_HandSolder, F.Cu at (161.0, 116.1)
- added C24: 100n, Capacitor_SMD:C_1206_3216Metric_Pad1.33x1.80mm_HandSolder, F.Cu at (157.2, 115.7)
- added C25: 100n, Capacitor_SMD:C_1206_3216Metric_Pad1.33x1.80mm_HandSolder, F.Cu at (229.9, 80.5)
- added C26: 100n, Capacitor_SMD:C_1206_3216Metric_Pad1.33x1.80mm_HandSolder, F.Cu at (142.3, 66.5)
- added C27: 100p, Capacitor_SMD:C_1206_3216Metric_Pad1.33x1.80mm_HandSolder, F.Cu at (236.5, 131.6)
- added C28: 100p, Capacitor_SMD:C_1206_3216Metric_Pad1.33x1.80mm_HandSolder, F.Cu at (230.8, 131.6)
- added C29: 10n, Capacitor_SMD:C_1206_3216Metric_Pad1.33x1.80mm_HandSolder, F.Cu at (226.6, 119.6)
- added C3: 4.7n, Capacitor_SMD:C_1206_3216Metric_Pad1.33x1.80mm_HandSolder, F.Cu at (187.6, 82.9)
- added C30: 10n, Capacitor_SMD:C_1206_3216Metric_Pad1.33x1.80mm_HandSolder, F.Cu at (241.8, 119.9)
- added C31: 22p, Capacitor_SMD:C_1206_3216Metric_Pad1.33x1.80mm_HandSolder, F.Cu at (179.4, 60.8)
- added C32: 22p, Capacitor_SMD:C_1206_3216Metric_Pad1.33x1.80mm_HandSolder, F.Cu at (202.3, 60.5)
- added C33: 22p, Capacitor_SMD:C_1206_3216Metric_Pad1.33x1.80mm_HandSolder, F.Cu at (168.0, 58.9)
- added C34: 100n, Capacitor_SMD:C_1206_3216Metric_Pad1.33x1.80mm_HandSolder, F.Cu at (264.2, 127.1)
- added C35: 100n, Capacitor_SMD:C_1206_3216Metric_Pad1.33x1.80mm_HandSolder, F.Cu at (260.3, 126.8)
- added C36: 100u, Capacitor_SMD:CP_Elec_8x10, F.Cu at (254.1, 71.0)
- added C37: 100n, Capacitor_SMD:C_1206_3216Metric_Pad1.33x1.80mm_HandSolder, F.Cu at (239.9, 75.4)
- added C38: 100n, Capacitor_SMD:C_1206_3216Metric_Pad1.33x1.80mm_HandSolder, F.Cu at (262.8, 74.8)
- added C39: 100n, Capacitor_SMD:C_1206_3216Metric_Pad1.33x1.80mm_HandSolder, F.Cu at (239.9, 79.3)
- added C4: 22p, Capacitor_SMD:C_1206_3216Metric_Pad1.33x1.80mm_HandSolder, F.Cu at (171.1, 76.8)
- added C40: 10u, Capacitor_SMD:CP_Elec_5x5.4, F.Cu at (247.2, 78.3)
- added C41: 10u, Capacitor_SMD:CP_Elec_5x5.4, F.Cu at (261.8, 81.5)
- added C42: 100n, Capacitor_SMD:C_1206_3216Metric_Pad1.33x1.80mm_HandSolder, F.Cu at (247.6, 85.6)
- added C43: 1000u, Capacitor_SMD:CP_Elec_8x10.5, F.Cu at (242.2, 67.8)
- added C44: 4.7n, Capacitor_SMD:C_1206_3216Metric_Pad1.33x1.80mm_HandSolder, F.Cu at (207.0, 133.2)
- added C45: 4.7n, Capacitor_SMD:C_1206_3216Metric_Pad1.33x1.80mm_HandSolder, F.Cu at (207.0, 129.4)
- added C46: 100n, Capacitor_SMD:C_1206_3216Metric_Pad1.33x1.80mm_HandSolder, F.Cu at (207.0, 125.6)
- added C47: 4.7n, Capacitor_SMD:C_1206_3216Metric_Pad1.33x1.80mm_HandSolder, F.Cu at (207.0, 121.8)
- added C48: 100n, Capacitor_SMD:C_1206_3216Metric_Pad1.33x1.80mm_HandSolder, F.Cu at (207.0, 118.0)
- added C49: 4.7n, Capacitor_SMD:C_1206_3216Metric_Pad1.33x1.80mm_HandSolder, F.Cu at (207.0, 114.2)
- added C5: 4.7n, Capacitor_SMD:C_1206_3216Metric_Pad1.33x1.80mm_HandSolder, F.Cu at (187.9, 79.1)
- added C50: 100n, Capacitor_SMD:C_1206_3216Metric_Pad1.33x1.80mm_HandSolder, F.Cu at (207.0, 110.4)
- added C51: 1u, Capacitor_SMD:CP_Elec_5x5.4, F.Cu at (129.0, 111.0)
- added C52: 100n, Capacitor_SMD:C_1206_3216Metric_Pad1.33x1.80mm_HandSolder, F.Cu at (140.7, 126.9)
- added C53: 22p, Capacitor_SMD:C_1206_3216Metric_Pad1.33x1.80mm_HandSolder, F.Cu at (130.3, 133.2)
- added C54: 22p, Capacitor_SMD:C_1206_3216Metric_Pad1.33x1.80mm_HandSolder, F.Cu at (136.0, 133.2)
- added C55: 1u, Capacitor_SMD:CP_Elec_5x5.4, F.Cu at (117.2, 141.8)
- added C56: 1u, Capacitor_SMD:CP_Elec_5x5.4, F.Cu at (107.4, 121.8)
- added C57: 1u, Capacitor_SMD:CP_Elec_5x5.4, F.Cu at (108.7, 142.8)
- added C58: 1u, Capacitor_SMD:CP_Elec_5x5.4, F.Cu at (107.0, 112.6)
- added C59: 10u, Capacitor_SMD:CP_Elec_5x5.4, F.Cu at (50.8, 128.8)
- added C6: 100n, Capacitor_SMD:C_1206_3216Metric_Pad1.33x1.80mm_HandSolder, F.Cu at (146.1, 92.4)
- added C60: 22p, Capacitor_SMD:C_1206_3216Metric_Pad1.33x1.80mm_HandSolder, F.Cu at (75.3, 136.4)
- added C61: 22p, Capacitor_SMD:C_1206_3216Metric_Pad1.33x1.80mm_HandSolder, F.Cu at (75.3, 142.8)
- added C62: 10u, Capacitor_SMD:CP_Elec_5x5.4, F.Cu at (60.0, 130.7)
- added C63: 100n, Capacitor_SMD:C_1206_3216Metric_Pad1.33x1.80mm_HandSolder, F.Cu at (43.2, 126.2)
- added C64: 47u, Capacitor_SMD:CP_Elec_6.3x5.8, F.Cu at (37.0, 118.6)
- added C65: 10u, Capacitor_SMD:CP_Elec_5x5.4, F.Cu at (60.0, 123.1)
- added C66: 10u, Capacitor_SMD:CP_Elec_5x5.4, F.Cu at (35.3, 139.9)
- added C67: 1u, Capacitor_SMD:CP_Elec_5x5.4, F.Cu at (86.1, 142.2)
- added C68: 1n, Capacitor_SMD:C_1206_3216Metric_Pad1.33x1.80mm_HandSolder, F.Cu at (70.8, 136.1)
- added C69: 10u, Capacitor_SMD:C_1206_3216Metric_Pad1.33x1.80mm_HandSolder, F.Cu at (67.0, 132.2)
- added C7: 100n, Capacitor_SMD:C_1206_3216Metric_Pad1.33x1.80mm_HandSolder, F.Cu at (146.1, 96.2)
- added C70: 68n, Capacitor_SMD:C_1206_3216Metric_Pad1.33x1.80mm_HandSolder, F.Cu at (51.5, 122.4)
- added C71: 1u, Capacitor_SMD:CP_Elec_5x5.4, F.Cu at (95.2, 143.0)
- added C72: 1u, Capacitor_SMD:CP_Elec_5x5.4, F.Cu at (94.9, 135.8)
- added C73: 10u, Capacitor_SMD:C_1206_3216Metric_Pad1.33x1.80mm_HandSolder, F.Cu at (45.1, 117.4)
- added C74: 1n, Capacitor_SMD:C_1206_3216Metric_Pad1.33x1.80mm_HandSolder, F.Cu at (51.8, 117.4)
- added C75: 1u, Capacitor_SMD:CP_Elec_5x5.4, F.Cu at (94.9, 128.1)
- added C76: 4.7u, Capacitor_SMD:CP_Elec_4x5.4, F.Cu at (95.3, 121.2)
- added C77: 10u, Capacitor_SMD:CP_Elec_5x5.4, F.Cu at (94.9, 114.2)
- added C78: 22p, Capacitor_SMD:C_1206_3216Metric_Pad1.33x1.80mm_HandSolder, F.Cu at (88.6, 113.0)
- added C79: 10u, Capacitor_SMD:CP_Elec_5x5.4, F.Cu at (60.0, 114.8)
- added C8: 22p, Capacitor_SMD:C_1206_3216Metric_Pad1.33x1.80mm_HandSolder, F.Cu at (145.4, 88.6)
- added C80: 22p, Capacitor_SMD:C_1206_3216Metric_Pad1.33x1.80mm_HandSolder, F.Cu at (88.6, 106.7)
- added C81: 1u, Capacitor_SMD:CP_Elec_5x5.4, F.Cu at (60.0, 106.6)
- added C82: 1u, Capacitor_SMD:CP_Elec_5x5.4, F.Cu at (94.9, 106.6)
- added C83: 4.7n, Capacitor_SMD:C_1206_3216Metric_Pad1.33x1.80mm_HandSolder, F.Cu at (60.5, 53.2)
- added C84: 4.7n, Capacitor_SMD:C_1206_3216Metric_Pad1.33x1.80mm_HandSolder, F.Cu at (38.6, 57.7)
- added C85: 4.7n, Capacitor_SMD:C_1206_3216Metric_Pad1.33x1.80mm_HandSolder, F.Cu at (33.8, 58.9)
- added C86: 4.7n, Capacitor_SMD:C_1206_3216Metric_Pad1.33x1.80mm_HandSolder, F.Cu at (45.0, 54.2)
- added C87: 10u, Capacitor_SMD:CP_Elec_5x5.4, F.Cu at (82.1, 57.7)
- added C9: 4.7n, Capacitor_SMD:C_1206_3216Metric_Pad1.33x1.80mm_HandSolder, F.Cu at (187.9, 75.3)
- added D1: 1N4148, Diode_SMD:D_SOD-523, F.Cu at (145.7, 84.2)
- added D10: 1N4148, Diode_SMD:D_SOD-523, F.Cu at (186.5, 114.8)
- added D11: 1N4148, Diode_SMD:D_SOD-523, F.Cu at (186.5, 117.4)
- added D12: 1N4148, Diode_SMD:D_SOD-523, F.Cu at (185.8, 132.0)
- added D13: 1N4148, Diode_SMD:D_SOD-523, F.Cu at (190.8, 121.2)
- added D14: 1N4148, Diode_SMD:D_SOD-523, F.Cu at (190.9, 125.0)
- added D15: 1N4148, Diode_SMD:D_SOD-523, F.Cu at (190.8, 112.3)
- added D16: 1N4148, Diode_SMD:D_SOD-523, F.Cu at (190.9, 114.8)
- added D17: 1N4148, Diode_SMD:D_SOD-523, F.Cu at (190.8, 109.7)
- added D18: 1N4148, Diode_SMD:D_SOD-523, F.Cu at (190.9, 118.6)
- added D19: Orange, MyFootprints:2-pin JST LED, F.Cu at (206.8, 138.9)
- added D2: 1N4148, Diode_SMD:D_SOD-523, F.Cu at (174.6, 90.5)
- added D20: Orange, MyFootprints:2-pin JST LED, F.Cu at (197.3, 138.9)
- added D21: Green, MyFootprints:2-pin JST LED, F.Cu at (187.7, 138.9)
- added D22: 1N4148, Diode_SMD:D_SOD-523, F.Cu at (213.1, 133.2)
- added D23: Green, MyFootprints:2-pin JST LED, F.Cu at (137.5, 119.9)
- added D24: Green, MyFootprints:2-pin JST LED, F.Cu at (137.5, 110.4)
- added D25: 1N4148, Diode_SMD:D_SOD-523, F.Cu at (115.1, 116.3)
- added D26: D_Zener, Package_TO_SOT_SMD:SOT-23_Handsoldering, F.Cu at (129.0, 143.6)
- added D27: D_Zener, Package_TO_SOT_SMD:SOT-23_Handsoldering, F.Cu at (135.6, 143.6)
- added D28: D_Zener, Package_TO_SOT_SMD:SOT-23_Handsoldering, F.Cu at (129.3, 138.3)
- added D29: D_Zener, Package_TO_SOT_SMD:SOT-23_Handsoldering, F.Cu at (135.6, 138.3)
- added D3: 1N4148, Diode_SMD:D_SOD-523, F.Cu at (170.5, 96.1)
- added D30: 1N4148, Diode_SMD:D_SOD-523, F.Cu at (112.1, 115.5)
- added D31: 1N4148, Diode_SMD:D_SOD-523, F.Cu at (41.0, 110.4)
- added D32: 1N4148, Diode_SMD:D_SOD-523, F.Cu at (41.0, 106.6)
- added D33: 1N4148, Diode_SMD:D_SOD-523, F.Cu at (38.4, 110.4)
- added D34: 1N4148, Diode_SMD:D_SOD-523, F.Cu at (38.4, 106.6)
- added D35: 1N4148, Diode_SMD:D_SOD-523, F.Cu at (55.7, 64.6)
- added D36: 1N4148, Diode_SMD:D_SOD-523, F.Cu at (47.8, 68.4)
- added D4: LED, MyFootprints:2-pin JST LED, F.Cu at (154.7, 124.3)
- added D5: LED, MyFootprints:2-pin JST LED, F.Cu at (154.7, 135.1)
- added D6: SK38, Diode_SMD:D_SMB, F.Cu at (263.1, 64.0)
- added D7: SK38, Diode_SMD:D_SMB, F.Cu at (263.1, 55.8)
- added D8: SK38, Diode_SMD:D_SMB, F.Cu at (250.4, 60.6)
- added D9: 1N4148, Diode_SMD:D_SOD-523, F.Cu at (186.5, 112.3)
- added J1: ICSP, MyFootprints:2x3_ISP_header, F.Cu at (181.9, 91.1)
- added J10: UART, Connector_PinHeader_2.54mm:PinHeader_1x03_P2.54mm_Vertical, F.Cu at (230.2, 58.2)
- added J11: HDMI_A, MyFootprints:HDMI_A_Kycon_KDMIX-SL1-NS-WS-B15_VerticalRightAngle, F.Cu at (227.1, 41.2)
- added J3: Paddle In, MyFootprints:3,5mm Jack Panel Socket 3-pole Switch large, F.Cu at (234.5, 146.6)
- added J4: USB Internal Conn, Connector_PinHeader_2.54mm:PinHeader_2x02_P2.54mm_Vertical, F.Cu at (191.5, 61.8)
- added J5: DB25_Receptacle_MountingHoles, Connector_Dsub:DSUB-25_Female_Horizontal_P2.77x2.84mm_EdgePinOffset4.94mm_Housed_MountingHolesOffset4.94mm, F.Cu at (174.4, 46.2)
- added J6: Micro_SD_Card_Det2, Connector_Card:microSD_HC_Hirose_DM3AT-SF-PEJM5, F.Cu at (256.5, 139.6)
- added J7: Barrel_Jack_Switch, MyFootprints:BarrelJack_Horizontal, F.Cu at (261.2, 49.1)
- added J8: Conn_02x04_Odd_Even, Connector_PinHeader_2.54mm:PinHeader_2x04_P2.54mm_Vertical, F.Cu at (116.6, 132.6)
- added J9: Mic In, MyFootprints:3,5mm Jack Panel Socket 3-pole Switch large, F.Cu at (78.6, 40.2)
- added JP1: Self Reset On, Connector_PinHeader_2.54mm:PinHeader_1x02_P2.54mm_Vertical, F.Cu at (140.0, 91.8)
- added JP2: Auro Reset On, Connector_PinHeader_2.54mm:PinHeader_1x02_P2.54mm_Vertical, F.Cu at (140.0, 96.2)
- added JP3: DTR to CW / FSK, MyFootprints:Jumper_1x03_P2.54mm_large, F.Cu at (173.7, 122.4)
- added JP4: AGND-GND, Connector_PinHeader_2.54mm:PinHeader_1x02_P2.54mm_Vertical, F.Cu at (227.7, 68.5)
- added JP5: ICOM / Other, MyFootprints:Jumper_1x03_P2.54mm_large, F.Cu at (162.3, 55.4)
- added JP6: REL - ULN, MyFootprints:Jumper_1x03_P2.54mm_large, F.Cu at (213.1, 124.3)
- added JP7: DC to Mic, Connector_PinHeader_2.54mm:PinHeader_1x02_P2.54mm_Vertical, F.Cu at (74.2, 55.8)
- added K1: G5V-1, Relay_THT:Relay_SPDT_Omron_G5V-1, F.Cu at (212.0, 109.2)
- added K2: G5V-1, Relay_THT:Relay_SPDT_Omron_G5V-1, F.Cu at (60.3, 58.4)
- added K3: G5V-1, Relay_THT:Relay_SPDT_Omron_G5V-1, F.Cu at (42.3, 62.9)
- added L10: L, Inductor_SMD:L_1206_3216Metric_Pad1.22x1.90mm_HandSolder, F.Cu at (206.1, 60.1)
- added L11: 10uH, Inductor_SMD:L_1206_3216Metric_Pad1.22x1.90mm_HandSolder, F.Cu at (179.4, 52.7)
- added L12: 10uH, Inductor_SMD:L_1206_3216Metric_Pad1.22x1.90mm_HandSolder, F.Cu at (183.3, 52.7)
- added L13: 10uH, Inductor_SMD:L_1206_3216Metric_Pad1.22x1.90mm_HandSolder, F.Cu at (187.1, 52.7)
- added L14: 10uH, Inductor_SMD:L_1206_3216Metric_Pad1.22x1.90mm_HandSolder, F.Cu at (190.9, 52.7)
- added L15: 10uH, Inductor_SMD:L_1206_3216Metric_Pad1.22x1.90mm_HandSolder, F.Cu at (194.7, 52.7)
- added L16: 10uH, Inductor_SMD:L_1206_3216Metric_Pad1.22x1.90mm_HandSolder, F.Cu at (198.5, 52.7)
- added L17: 10uH, Inductor_SMD:L_1206_3216Metric_Pad1.22x1.90mm_HandSolder, F.Cu at (202.3, 52.7)
- added L18: L, Inductor_SMD:L_1206_3216Metric_Pad1.22x1.90mm_HandSolder, F.Cu at (171.8, 52.7)
- added L19: 10uH, Inductor_SMD:L_1206_3216Metric_Pad1.22x1.90mm_HandSolder, F.Cu at (206.1, 52.7)
- added L20: 10uH, Inductor_SMD:L_1206_3216Metric_Pad1.22x1.90mm_HandSolder, F.Cu at (209.9, 52.7)
- added L21: 10uH, Inductor_SMD:L_1206_3216Metric_Pad1.22x1.90mm_HandSolder, F.Cu at (213.7, 52.7)
- added L22: L, Inductor_SMD:L_1206_3216Metric_Pad1.22x1.90mm_HandSolder, F.Cu at (168.0, 52.7)
- added L23: 10uH, Inductor_SMD:L_1206_3216Metric_Pad1.22x1.90mm_HandSolder, F.Cu at (217.6, 52.7)
- added L24: 100uH, Inductor_SMD:L_1206_3216Metric_Pad1.22x1.90mm_HandSolder, F.Cu at (262.7, 71.0)
- added L25: 100uH, Inductor_SMD:L_1206_3216Metric_Pad1.22x1.90mm_HandSolder, F.Cu at (245.3, 59.6)
- added L26: L, Inductor_SMD:L_1206_3216Metric_Pad1.22x1.90mm_HandSolder, F.Cu at (121.7, 111.6)
- added L27: L, Inductor_SMD:L_1206_3216Metric_Pad1.22x1.90mm_HandSolder, F.Cu at (89.0, 101.3)
- added L28: 10uH, Inductor_SMD:L_1206_3216Metric_Pad1.22x1.90mm_HandSolder, F.Cu at (66.5, 53.2)
- added L29: 10uH, Inductor_SMD:L_1206_3216Metric_Pad1.22x1.90mm_HandSolder, F.Cu at (33.8, 53.2)
- added L30: 10uH, Inductor_SMD:L_1206_3216Metric_Pad1.22x1.90mm_HandSolder, F.Cu at (40.3, 53.2)
- added L31: 10uH, Inductor_SMD:L_1206_3216Metric_Pad1.22x1.90mm_HandSolder, F.Cu at (54.5, 53.2)
- added L5: L, Inductor_SMD:L_1206_3216Metric_Pad1.22x1.90mm_HandSolder, F.Cu at (155.3, 110.0)
- added L6: 10uH, Inductor_SMD:L_1206_3216Metric_Pad1.22x1.90mm_HandSolder, F.Cu at (242.5, 143.0)
- added L7: 10uH, Inductor_SMD:L_1206_3216Metric_Pad1.22x1.90mm_HandSolder, F.Cu at (226.0, 143.2)
- added L8: 10uH, Inductor_SMD:L_1206_3216Metric_Pad1.22x1.90mm_HandSolder, F.Cu at (175.6, 52.7)
- added L9: L, Inductor_SMD:L_1206_3216Metric_Pad1.22x1.90mm_HandSolder, F.Cu at (187.1, 60.8)
- added Q1: BC856BDW1, Package_TO_SOT_SMD:SOT-363_SC-70-6_Handsoldering, F.Cu at (170.5, 139.0)
- added Q2: BSS84, Package_TO_SOT_SMD:SOT-23, F.Cu at (165.8, 138.6)
- added Q3: BC817, Package_TO_SOT_SMD:SOT-23-3, F.Cu at (166.1, 143.9)
- added Q4: BC817, Package_TO_SOT_SMD:SOT-23-3, F.Cu at (36.7, 125.6)
- added Q5: BC817, Package_TO_SOT_SMD:SOT-23-3, F.Cu at (55.1, 59.6)
- added Q6: BC856B, Package_TO_SOT_SMD:SOT-23-3, F.Cu at (48.4, 64.0)
- added R1: 220R, Resistor_SMD:R_1206_3216Metric_Pad1.30x1.75mm_HandSolder, F.Cu at (181.9, 86.7)
- added R10: 1k5, Resistor_SMD:R_1206_3216Metric_Pad1.30x1.75mm_HandSolder, F.Cu at (174.3, 95.2)
- added R14: 24R, Resistor_SMD:R_1206_3216Metric_Pad1.30x1.75mm_HandSolder, F.Cu at (88.9, 92.5)
- added R15: 24R, Resistor_SMD:R_1206_3216Metric_Pad1.30x1.75mm_HandSolder, F.Cu at (77.1, 92.5)
- added R16: 1k5, Resistor_SMD:R_1206_3216Metric_Pad1.30x1.75mm_HandSolder, F.Cu at (82.8, 87.4)
- added R17: 1k5, Resistor_SMD:R_1206_3216Metric_Pad1.30x1.75mm_HandSolder, F.Cu at (71.4, 92.5)
- added R18: 1M, Resistor_SMD:R_1206_3216Metric_Pad1.30x1.75mm_HandSolder, F.Cu at (70.1, 81.1)
- added R19: 27R, Resistor_SMD:R_1206_3216Metric_Pad1.30x1.75mm_HandSolder, F.Cu at (173.1, 110.4)
- added R2: 1M, Resistor_SMD:R_1206_3216Metric_Pad1.30x1.75mm_HandSolder, F.Cu at (167.3, 76.8)
- added R20: 1k5, Resistor_SMD:R_1206_3216Metric_Pad1.30x1.75mm_HandSolder, F.Cu at (169.3, 116.1)
- added R21: 27R, Resistor_SMD:R_1206_3216Metric_Pad1.30x1.75mm_HandSolder, F.Cu at (169.3, 110.4)
- added R22: 1k5, Resistor_SMD:R_1206_3216Metric_Pad1.30x1.75mm_HandSolder, F.Cu at (165.5, 115.8)
- added R23: 1k5, Resistor_SMD:R_1206_3216Metric_Pad1.30x1.75mm_HandSolder, F.Cu at (165.5, 110.4)
- added R24: 1k5, Resistor_SMD:R_1206_3216Metric_Pad1.30x1.75mm_HandSolder, F.Cu at (170.6, 144.7)
- added R25: 1k5, Resistor_SMD:R_1206_3216Metric_Pad1.30x1.75mm_HandSolder, F.Cu at (170.6, 133.2)
- added R26: 10k, Resistor_SMD:R_1206_3216Metric_Pad1.30x1.75mm_HandSolder, F.Cu at (166.7, 132.9)
- added R27: 4k7, Resistor_SMD:R_1206_3216Metric_Pad1.30x1.75mm_HandSolder, F.Cu at (161.0, 138.6)
- added R28: 10k, Resistor_SMD:R_1206_3216Metric_Pad1.30x1.75mm_HandSolder, F.Cu at (174.4, 132.9)
- added R29: 470R, Resistor_SMD:R_1206_3216Metric_Pad1.30x1.75mm_HandSolder, F.Cu at (150.9, 115.1)
- added R3: 220R, Resistor_SMD:R_1206_3216Metric_Pad1.30x1.75mm_HandSolder, F.Cu at (181.9, 82.9)
- added R30: 470R, Resistor_SMD:R_1206_3216Metric_Pad1.30x1.75mm_HandSolder, F.Cu at (151.8, 140.8)
- added R31: 1k6, Resistor_SMD:R_1206_3216Metric_Pad1.30x1.75mm_HandSolder, F.Cu at (174.4, 138.9)
- added R32: 1k, Resistor_SMD:R_1206_3216Metric_Pad1.30x1.75mm_HandSolder, F.Cu at (161.0, 132.9)
- added R33: 4k7, Resistor_SMD:R_1206_3216Metric_Pad1.30x1.75mm_HandSolder, F.Cu at (224.2, 84.3)
- added R34: 10k, Resistor_SMD:R_1206_3216Metric_Pad1.30x1.75mm_HandSolder, F.Cu at (229.9, 84.3)
- added R35: 10k, Resistor_SMD:R_1206_3216Metric_Pad1.30x1.75mm_HandSolder, F.Cu at (224.2, 80.5)
- added R36: 470R, Resistor_SMD:R_1206_3216Metric_Pad1.30x1.75mm_HandSolder, F.Cu at (242.5, 136.9)
- added R37: 470R, Resistor_SMD:R_1206_3216Metric_Pad1.30x1.75mm_HandSolder, F.Cu at (226.0, 137.0)
- added R38: 10k, Resistor_SMD:R_1206_3216Metric_Pad1.30x1.75mm_HandSolder, F.Cu at (231.4, 114.5)
- added R39: 10k, Resistor_SMD:R_1206_3216Metric_Pad1.30x1.75mm_HandSolder, F.Cu at (231.4, 110.7)
- added R4: 220R, Resistor_SMD:R_1206_3216Metric_Pad1.30x1.75mm_HandSolder, F.Cu at (182.2, 79.1)
- added R40: 15k, Resistor_SMD:R_1206_3216Metric_Pad1.30x1.75mm_HandSolder, F.Cu at (234.7, 93.2)
- added R41: 1k5, Resistor_SMD:R_1206_3216Metric_Pad1.30x1.75mm_HandSolder, F.Cu at (243.6, 93.2)
- added R42: 1k5, Resistor_SMD:R_1206_3216Metric_Pad1.30x1.75mm_HandSolder, F.Cu at (253.4, 93.2)
- added R43: 10k, Resistor_SMD:R_1206_3216Metric_Pad1.30x1.75mm_HandSolder, F.Cu at (237.1, 110.7)
- added R44: 1k5, Resistor_SMD:R_1206_3216Metric_Pad1.30x1.75mm_HandSolder, F.Cu at (262.3, 93.2)
- added R45: 10k, Resistor_SMD:R_1206_3216Metric_Pad1.30x1.75mm_HandSolder, F.Cu at (237.1, 114.5)
- added R46: 27R, Resistor_SMD:R_1206_3216Metric_Pad1.30x1.75mm_HandSolder, F.Cu at (175.6, 60.8)
- added R47: 27R, Resistor_SMD:R_1206_3216Metric_Pad1.30x1.75mm_HandSolder, F.Cu at (213.7, 59.6)
- added R48: 1k5, Resistor_SMD:R_1206_3216Metric_Pad1.30x1.75mm_HandSolder, F.Cu at (183.3, 60.8)
- added R49: 1k5, Resistor_SMD:R_1206_3216Metric_Pad1.30x1.75mm_HandSolder, F.Cu at (209.9, 60.2)
- added R5: 220R, Resistor_SMD:R_1206_3216Metric_Pad1.30x1.75mm_HandSolder, F.Cu at (182.2, 75.3)
- added R50: 15k, Resistor_SMD:R_1206_3216Metric_Pad1.30x1.75mm_HandSolder, F.Cu at (198.5, 60.2)
- added R51: 1k5, Resistor_SMD:R_1206_3216Metric_Pad1.30x1.75mm_HandSolder, F.Cu at (171.8, 58.9)
- added R52: 100k, Resistor_SMD:R_1206_3216Metric_Pad1.30x1.75mm_HandSolder, F.Cu at (262.5, 121.7)
- added R53: 470R, Resistor_SMD:R_1206_3216Metric_Pad1.30x1.75mm_HandSolder, F.Cu at (187.1, 124.0)
- added R54: 470R, Resistor_SMD:R_1206_3216Metric_Pad1.30x1.75mm_HandSolder, F.Cu at (190.0, 128.1)
- added R55: 470R, Resistor_SMD:R_1206_3216Metric_Pad1.30x1.75mm_HandSolder, F.Cu at (190.0, 132.0)
- added R56: 1k5, Resistor_SMD:R_1206_3216Metric_Pad1.30x1.75mm_HandSolder, F.Cu at (130.3, 125.6)
- added R57: 15k, Resistor_SMD:R_1206_3216Metric_Pad1.30x1.75mm_HandSolder, F.Cu at (141.3, 132.6)
- added R58: 15k, Resistor_SMD:R_1206_3216Metric_Pad1.30x1.75mm_HandSolder, F.Cu at (136.0, 129.4)
- added R59: 27R, Resistor_SMD:R_1206_3216Metric_Pad1.30x1.75mm_HandSolder, F.Cu at (130.3, 129.4)
- added R6: 10k, Resistor_SMD:R_1206_3216Metric_Pad1.30x1.75mm_HandSolder, F.Cu at (146.1, 81.6)
- added R60: 27R, Resistor_SMD:R_1206_3216Metric_Pad1.30x1.75mm_HandSolder, F.Cu at (136.0, 125.6)
- added R61: 470R, Resistor_SMD:R_1206_3216Metric_Pad1.30x1.75mm_HandSolder, F.Cu at (130.3, 121.8)
- added R62: 470R, Resistor_SMD:R_1206_3216Metric_Pad1.30x1.75mm_HandSolder, F.Cu at (130.3, 118.0)
- added R63: 4k7, Resistor_SMD:R_1206_3216Metric_Pad1.30x1.75mm_HandSolder, F.Cu at (115.0, 111.6)
- added R64: 1k, Resistor_SMD:R_1206_3216Metric_Pad1.30x1.75mm_HandSolder, F.Cu at (114.4, 121.2)
- added R65: 220R, Resistor_SMD:R_1206_3216Metric_Pad1.30x1.75mm_HandSolder, F.Cu at (123.3, 143.4)
- added R66: 220R, Resistor_SMD:R_1206_3216Metric_Pad1.30x1.75mm_HandSolder, F.Cu at (123.3, 138.0)
- added R67: 27R, Resistor_SMD:R_1206_3216Metric_Pad1.30x1.75mm_HandSolder, F.Cu at (80.1, 138.0)
- added R68: 4k7, Resistor_SMD:R_1206_3216Metric_Pad1.30x1.75mm_HandSolder, F.Cu at (42.9, 130.7)
- added R69: 100k, Resistor_SMD:R_1206_3216Metric_Pad1.30x1.75mm_HandSolder, F.Cu at (37.0, 130.1)
- added R7: 15k, Resistor_SMD:R_1206_3216Metric_Pad1.30x1.75mm_HandSolder, F.Cu at (159.1, 76.5)
- added R70: 470R, Resistor_SMD:R_1206_3216Metric_Pad1.30x1.75mm_HandSolder, F.Cu at (40.7, 101.5)
- added R71: 27R, Resistor_SMD:R_1206_3216Metric_Pad1.30x1.75mm_HandSolder, F.Cu at (86.4, 134.2)
- added R72: 15k, Resistor_SMD:R_1206_3216Metric_Pad1.30x1.75mm_HandSolder, F.Cu at (70.8, 142.8)
- added R73: 1k5, Resistor_SMD:R_1206_3216Metric_Pad1.30x1.75mm_HandSolder, F.Cu at (80.1, 134.2)
- added R74: 15k, Resistor_SMD:R_1206_3216Metric_Pad1.30x1.75mm_HandSolder, F.Cu at (80.3, 143.1)
- added R75: 100k, Resistor_SMD:R_1206_3216Metric_Pad1.30x1.75mm_HandSolder, F.Cu at (34.0, 111.0)
- added R76: 4k7, Resistor_SMD:R_1206_3216Metric_Pad1.30x1.75mm_HandSolder, F.Cu at (67.3, 125.3)
- added R77: 4k7, Resistor_SMD:R_1206_3216Metric_Pad1.30x1.75mm_HandSolder, F.Cu at (67.7, 115.8)
- added R78: 4k7, Resistor_SMD:R_1206_3216Metric_Pad1.30x1.75mm_HandSolder, F.Cu at (67.7, 107.5)
- added R79: 470R, Resistor_SMD:R_1206_3216Metric_Pad1.30x1.75mm_HandSolder, F.Cu at (45.1, 121.2)
- added R8: 1k5, Resistor_SMD:R_1206_3216Metric_Pad1.30x1.75mm_HandSolder, F.Cu at (162.9, 76.5)
- added R80: 1k, Resistor_SMD:R_1206_3216Metric_Pad1.30x1.75mm_HandSolder, F.Cu at (62.9, 100.8)
- added R81: 1M, Resistor_SMD:R_1206_3216Metric_Pad1.30x1.75mm_HandSolder, F.Cu at (82.6, 100.8)
- added R82: 4k7, Resistor_SMD:R_1206_3216Metric_Pad1.30x1.75mm_HandSolder, F.Cu at (69.9, 100.8)
- added R83: 10k, Resistor_SMD:R_1206_3216Metric_Pad1.30x1.75mm_HandSolder, F.Cu at (52.9, 68.5)
- added R84: 1k5, Resistor_SMD:R_1206_3216Metric_Pad1.30x1.75mm_HandSolder, F.Cu at (50.0, 54.2)
- added R85: 1k5, Resistor_SMD:R_1206_3216Metric_Pad1.30x1.75mm_HandSolder, F.Cu at (82.1, 63.5)
- added R9: 1k5, Resistor_SMD:R_1206_3216Metric_Pad1.30x1.75mm_HandSolder, F.Cu at (171.1, 91.4)
- added RV1: 10k, MyFootprints:3-pin JST Potentiometer, F.Cu at (56.2, 80.5)
- added RV2: 10k, MyFootprints:3-pin JST Potentiometer, F.Cu at (56.2, 92.0)
- added RV3: 18VDC, Varistor:RV_Disc_D12mm_W3.9mm_P7.5mm, F.Cu at (256.0, 62.0)
- added RV4: 10k log, MyFootprints:3-pin JST Potentiometer, F.Cu at (47.3, 137.7)
- added RV5: 10k, MyFootprints:3-pin JST Potentiometer, F.Cu at (75.4, 65.3)
- added SW1: RotaryEncoder, MyFootprints:3-pin JST Rotary Encoder, F.Cu at (231.8, 119.9)
- added T1: Transformer_1P_1S, MyFootprints:Audio Transformer Bourns SM-LP-5001, F.Cu at (53.8, 138.3)
- added T2: Transformer_1P_1S, MyFootprints:Audio Transformer Bourns SM-LP-5001, F.Cu at (47.3, 112.8)
- added U1: Reset, MyFootprints:2-pin JST Switch, F.Cu at (138.8, 83.6)
- added U10: M1, MyFootprints:2-pin JST Switch, F.Cu at (242.3, 98.9)
- added U11: M2, MyFootprints:2-pin JST Switch, F.Cu at (251.8, 98.9)
- added U12: Mode, MyFootprints:2-pin JST Switch, F.Cu at (261.4, 98.9)
- added U13: LSF0102, Package_TO_SOT_SMD:SOT-23W_Handsoldering, F.Cu at (255.6, 126.6)
- added U14: LSF0102, Package_TO_SOT_SMD:SOT-23W_Handsoldering, F.Cu at (250.2, 126.6)
- added U15: LM2576HVS-5, Package_TO_SOT_SMD:TO-263-5_TabPin3, F.Cu at (247.0, 45.9)
- added U16: L78L33_SOT89, Package_TO_SOT_SMD:SOT-89-3_Handsoldering, F.Cu at (254.8, 81.8)
- added U17: ULN2803A, MyFootprints:DIP-18_W7.62mm w socket, F.Cu at (194.7, 112.3)
- added U18: FT232RL, Package_SO:SSOP-28_5.3x10.2mm_P0.65mm, F.Cu at (122.3, 121.2)
- added U19: MAX232, Package_SO:SOIC-16_3.9x9.9mm_P1.27mm, F.Cu at (108.3, 131.3)
- added U2: ATmega2560-16A, Package_QFP:TQFP-100_14x14mm_P0.5mm, F.Cu at (159.1, 88.6)
- added U20: Vol -, MyFootprints:2-pin JST Switch, F.Cu at (73.4, 125.6)
- added U21: Vol +, MyFootprints:2-pin JST Switch, F.Cu at (73.4, 116.1)
- added U22: Mute, MyFootprints:2-pin JST Switch, F.Cu at (73.4, 106.6)
- added U23: PCM2904, Package_SO:SSOP-28_5.3x10.2mm_P0.65mm, F.Cu at (85.0, 123.3)
- added U24: 2 x RCA Jack, MyFootprints:pro-signal PSG01550 Dual 2× RCA Phono SocketRight Angle PCB, F.Cu at (63.4, 45.0)
- added U25: 2 x RCA Jack, MyFootprints:pro-signal PSG01550 Dual 2× RCA Phono SocketRight Angle PCB, F.Cu at (44.3, 45.0)
- added U5: TUSB2046B, Package_QFP:LQFP-32_7x7mm_P0.8mm, F.Cu at (85.1, 79.5)
- added U6: FT232RL, Package_SO:SSOP-28_5.3x10.2mm_P0.65mm, F.Cu at (164.8, 124.3)
- added U7: LCD_HD44780, MyFootprints:2 x 6-pin JST LCD HD44780 Stacked, F.Cu at (34.7, 89.9)
- added U8: USR-ES1 W5500, MyFootprints:USR-ES1 W5500, F.Cu at (131.8, 44.9)
- added U9: Set, MyFootprints:2-pin JST Switch, F.Cu at (232.8, 98.9)
- added Y1: 16MHz, Crystal:Crystal_SMD_HC49-SD, F.Cu at (175.6, 80.8)
- added Y2: 6MHz, Crystal:Crystal_SMD_HC49-SD, F.Cu at (75.8, 82.1)
- added Y3: 12 MHz, Crystal:Crystal_SMD_HC49-SD, F.Cu at (82.9, 109.5)
- moved R11 71.4 mm to (98.1, 48.1)
- moved U3 67.7 mm to (93.7, 53.5), turned to 90 degrees
- moved L1 66.9 mm to (98.1, 42.4)
- moved C14 65.4 mm to (105.1, 52.2)
- moved C15 65.4 mm to (122.9, 58.6)
- moved C16 65.4 mm to (122.9, 52.9)
- moved J2 65.4 mm to (107.7, 46.8)
- moved L2 65.4 mm to (98.5, 61.4)
- moved L3 65.4 mm to (98.8, 57.6)
- moved R12 65.4 mm to (104.2, 61.4)
- moved R13 65.4 mm to (104.5, 57.6)
- moved U4 65.4 mm to (114.2, 55.7)
- moved C13 65.1 mm to (98.8, 53.8)
- moved L4 64.6 mm to (119.7, 47.2), turned to -90 degrees
Routing:
- net AGNDC: track 4.57 -> 1623.4 mm, vias 0 -> 19
- net +5V: track 0.00 -> 948.7 mm, vias 0 -> 10
- net +3.3V: track 0.00 -> 479.6 mm, vias 0 -> 13
- net PA PTT Out: track 0.00 -> 275.5 mm, vias 0 -> 3
- net DTR: track 0.00 -> 256.9 mm, vias 0 -> 4
- net Interlock In: track 0.00 -> 245.5 mm, vias 0 -> 3
- net RX Audio GND: track 0.00 -> 230.0 mm, vias 0 -> 2
- net RX Audio: track 0.00 -> 226.8 mm, vias 0 -> 3
- net TX Audio GND: track 0.00 -> 224.6 mm, vias 0 -> 1
- net SEQ Out: track 0.00 -> 213.7 mm, vias 0 -> 3
- net Mic Out: track 0.00 -> 198.5 mm, vias 0 -> 1
- net Paddle Left: track 0.00 -> 179.9 mm, vias 0 -> 2
- net PTT from Foot: track 0.00 -> 170.9 mm, vias 0 -> 4
- net TX Audio: track 0.00 -> 160.4 mm, vias 0 -> 1
- net Paddle Right: track 0.00 -> 151.5 mm, vias 0 -> 4
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Other:
- board outline added: 239 x 110.5 mm
- board text added: "ACC"
- board text added: "Audio Switching"
- board text added: "Buttons"
- board text added: "Ethernet"
- board text added: "Micro SD"
- board text added: "Output"
- board text added: "Paddle Input"
- board text added: "USB Hub"
