File: KiCad/Open Interface III/Open Interface III.kicad_sch (KiCad schematic)
At the start: 0 parts

Commit message: OI III Schematics 0.1
Parts:
- added C1, C4, C8: 22p, symbol Device:C
- added C10, C11, C12, C6, C7: 100n, symbol Device:C
- added C2, C3, C5, C9: 4.7n, symbol Device:C
- added D1, D2, D3: 1N4148, symbol Diode:1N4148
- added J1: ICSP, symbol My_Parts:6-pin_ISP_connector
- added JP1: Self Reset On, symbol Jumper:Jumper_2_Bridged
- added JP2: Auro Reset On, symbol Jumper:Jumper_2_Bridged
- added R1, R3, R4, R5: 220R, symbol Device:R
- added R10, R8, R9: 1k5, symbol Device:R
- added R2: 1M, symbol Device:R
- added R6: 10k, symbol Device:R
- added R7: 15k, symbol Device:R
- added U1: Reset, symbol My_Parts:Switch
- added U2: ATmega2560-16A, symbol MCU_Microchip_ATmega:ATmega2560-16A
- added Y1: 16MHz, symbol Device:Crystal
Connections:
- new net: D3.2 (A), R10.2, U2.6 (PE4)
- new net: R1.1, U2.39 (PL4)
- new net: C7.1, JP2.1 (A)
- new net: C1.1, R2.1, U2.34 (XTAL1), Y1.1
- new net: C4.1, R2.2, U2.33 (XTAL2), Y1.2
- new net: R7.1, R8.1, U2.90 (PF7)
- new net: R5.1, U2.42 (PL7)
- new net: D2.2 (A), R9.2, U2.45 (PD2)
- new net: C10.2, C11.2, C12.2
- new net: C6.1, JP1.1 (A)
- new net: R4.1, U2.41 (PL6)
- new net: R3.1, U2.40 (PL5)
- new net +3.3V: U2.91 (PF6)
- new net +5V: C10.1, C11.1, C12.1, D1.1 (K), J1.2 (Pin_2), R10.1, R6.2, R9.1, U2.10 (VCC), U2.100 (AVCC), U2.31 (VCC), U2.61 (VCC), U2.80 (VCC)
- new net 10 (PWM): U2.23 (PB4)
- new net A0: U2.97 (PF0)
- new net A10: U2.87 (PK2)
- new net A11: U2.86 (PK3)
- new net A12: U2.85 (PK4)
- new net A13: U2.84 (PK5)
- new net A14: U2.83 (PK6)
- new net A15: U2.82 (PK7)
- new net A3: U2.94 (PF3)
- new net A4: U2.93 (PF4)
- new net A8: U2.89 (PK0)
- new net A9: U2.88 (PK1)
- new net AFSK: U2.71 (PA7)
- new net BCD1: C9.1, R5.2
- new net BCD2: C5.1, R4.2
- new net BCD3: C3.1, R3.2
- new net BCD4: C2.1, R1.2
- new net CW Tone: U2.1 (PG5)
- new net CW1: U2.56 (PC3)
- new net CW2: U2.55 (PC2)
- new net D11: U2.24 (PB5)
- new net D12: U2.25 (PB6)
- new net D13: U2.26 (PB7)
- new net D30: U2.60 (PC7)
- new net D32: U2.58 (PC5)
- new net D38: U2.50 (PD7)
- new net D46: U2.38 (PL3)
- new net D47: U2.37 (PL2)
- new net D48: U2.36 (PL1)
- new net D49: U2.35 (PL0)
- new net D5: U2.5 (PE3)
- new net D50 (MISO): J1.1 (Pin_1), U2.22 (PB3)
- new net D51 (MOSI): J1.4 (Pin_4), U2.21 (PB2)
- new net D52 (SCK): J1.3 (Pin_3), U2.20 (PB1)
- new net D53: U2.19 (PB0)
- new net DTR: JP2.2 (B)
- new net ENC B: U2.46 (PD3)
- new net Enc A: U2.76 (PA2)
- new net FSK Detector: U2.57 (PC4)
- new net FSK arduino: U2.77 (PA1)
- new net GND: C1.2, C2.2, C3.2, C4.2, C5.2, C8.2, C9.2, J1.6 (Pin_6), R8.2, U1.1 (Com), U2.11 (GND), U2.32 (GND), U2.62 (GND), U2.81 (GND), U2.99 (GND)
- new net Interlock In: D3.1 (K)
- new net LCD D4: U2.15 (PH3)
- new net LCD D5: U2.16 (PH4)
- new net LCD D6: U2.17 (PH5)
- new net LCD D7: U2.18 (PH6)
- new net LCD E: U2.53 (PC0)
- new net LCD RS: U2.95 (PF2)
- new net Mem: U2.96 (PF1)
- new net Menu: U2.54 (PC1)
- new net PA PTT: U2.59 (PC6)
- new net PTT 232: U2.7 (PE5)
- new net PTT from Foot: D2.1 (K)
- new net PTT1: U2.51 (PG0)
- new net PTT2: U2.78 (PA0)
- new net PTT3: U2.75 (PA3)
- new net Paddle Left: U2.74 (PA4)
- new net Paddle Right: U2.72 (PA6)
- new net Res Mega: C6.2, C7.2, C8.1, D1.2 (A), J1.5 (Pin_5), R6.1, U1.2 (NO), U2.30 (~{RESET})
- new net RxD: U2.3 (PE1)
- new net RxD2: U2.12 (PH0)
- new net RxD3: U2.63 (PJ0)
- new net SCL: U2.43 (PD0)
- new net SDA: U2.44 (PD1)
- new net SEQ: U2.52 (PG1)
- new net Self Res: JP1.2 (B), U2.70 (PG2)
- new net TxD: U2.2 (PE0)
- new net TxD2: U2.13 (PH1)
- new net TxD3: U2.64 (PJ1)
- new net Vin: R7.2
- new net WinKEY: U2.73 (PA5)
- new net microSD Plug: U2.92 (PF5)
Other:
- company: (none) -> Jonix
- title: (none) -> Open Interface III

Commit message: PCB 0.1, BOM
Parts:
- C1, C10, C11, C12, C2, C3, C4, C5, C6, C7, C8, C9: footprint (none) -> Capacitor_SMD:C_1206_3216Metric_Pad1.33x1.80mm_HandSolder
- D1, D2, D3: footprint (none) -> Diode_SMD:D_SOD-523
- J1: footprint (none) -> MyFootprints:2x3_ISP_header
- JP1, JP2: footprint (none) -> Connector_PinHeader_2.54mm:PinHeader_1x02_P2.54mm_Vertical
- R1, R10, R2, R3, R4, R5, R6, R7, R8, R9: footprint (none) -> Resistor_SMD:R_1206_3216Metric_Pad1.30x1.75mm_HandSolder
- U1: footprint (none) -> MyFootprints:2-pin JST Switch
- U2: footprint (none) -> Package_QFP:TQFP-100_14x14mm_P0.5mm
- Y1: footprint (none) -> Crystal:Crystal_SMD_HC49-SD
Changed lines of the file:
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@@
 			)
 		)
-		(property "Footprint" ""
+		(property "Footprint" "Diode_SMD:D_SOD-523"
 			(at 182.88 139.7 0)
 			(effects
@@
 			)
 		)
-		(property "Footprint" ""
+		(property "Footprint" "MyFootprints:2-pin JST Switch"
 			(at 35.56 53.34 0)
 			(effects
@@
 			)
 		)
-		(property "Footprint" ""
+		(property "Footprint" "Resistor_SMD:R_1206_3216Metric_Pad1.30x1.75mm_HandSolder"
 			(at 18.542 137.16 90)
 			(effects
@@
 			)
 		)
-		(property "Footprint" ""
+		(property "Footprint" "Capacitor_SMD:C_1206_3216Metric_Pad1.33x1.80mm_HandSolder"
 			(at 50.4952 50.8 0)
 			(effects
@@
 			)
 		)
-		(property "Footprint" ""
+		(property "Footprint" "Capacitor_SMD:C_1206_3216Metric_Pad1.33x1.80mm_HandSolder"
 			(at 41.6052 175.26 0)
 			(effects
@@
 			)
 		)
-		(property "Footprint" ""
+		(property "Footprint" "Capacitor_SMD:C_1206_3216Metric_Pad1.33x1.80mm_HandSolder"
 			(at 53.34 32.0548 0)
 			(effects
@@
 			)
 		)
-		(property "Footprint" ""
+		(property "Footprint" "Crystal:Crystal_SMD_HC49-SD"
 			(at 29.21 88.9 0)
 			(effects
@@
 			)
 		)
-		(property "Footprint" ""
+		(property "Footprint" "Connector_PinHeader_2.54mm:PinHeader_1x02_P2.54mm_Vertical"
 			(at 35.56 33.02 0)
 			(effects
@@
 			)
 		)
-		(property "Footprint" ""
+		(property "Footprint" "Resistor_SMD:R_1206_3216Metric_Pad1.30x1.75mm_HandSolder"
 			(at 170.942 129.54 90)
 			(effects
@@
 			)
 		)
-		(property "Footprint" ""
+		(property "Footprint" "Resistor_SMD:R_1206_3216Metric_Pad1.30x1.75mm_HandSolder"
 			(at 153.162 179.07 90)
 			(effects
@@
 			)
 		)
-		(property "Footprint" ""
+		(property "Footprint" "Resistor_SMD:R_1206_3216Metric_Pad1.30x1.75mm_HandSolder"
 			(at 77.47 23.368 90)
 			(effects
@@
 			)
 		)
-		(property "Footprint" ""
+		(property "Footprint" "Resistor_SMD:R_1206_3216Metric_Pad1.30x1.75mm_HandSolder"
 			(at 49.022 137.16 90)
 			(effects
@@
 			)
 		)
-		(property "Footprint" ""
+		(property "Footprint" "Resistor_SMD:R_1206_3216Metric_Pad1.30x1.75mm_HandSolder"
 			(at 170.942 101.6 90)
 			(effects
@@
 			)
 		)
-		(property "Footprint" ""
+		(property "Footprint" "Resistor_SMD:R_1206_3216Metric_Pad1.30x1.75mm_HandSolder"
 			(at 29.21 77.978 90)
 			(effects
@@
 			)
 		)
-		(property "Footprint" ""
+		(property "Footprint" "Capacitor_SMD:C_1206_3216Metric_Pad1.33x1.80mm_HandSolder"
 			(at 184.15 24.4348 0)
 			(effects
@@
 			)
 		)
-		(property "Footprint" ""
+		(property "Footprint" "Resistor_SMD:R_1206_3216Metric_Pad1.30x1.75mm_HandSolder"
 			(at 136.652 179.07 90)
 			(effects
@@
 			)
 		)
-		(property "Footprint" ""
+		(property "Footprint" "Connector_PinHeader_2.54mm:PinHeader_1x02_P2.54mm_Vertical"
 			(at 35.56 21.59 0)
 			(effects
@@
 			)
 		)
-		(property "Footprint" ""
+		(property "Footprint" "Capacitor_SMD:C_1206_3216Metric_Pad1.33x1.80mm_HandSolder"
 			(at 21.2852 101.6 0)
 			(effects
@@
 			)
 		)
-		(property "Footprint" ""
+		(property "Footprint" "Capacitor_SMD:C_1206_3216Metric_Pad1.33x1.80mm_HandSolder"
 			(at 39.0652 101.6 0)
 			(effects
@@
 			)
 		)
-		(property "Footprint" ""
+		(property "Footprint" "Resistor_SMD:R_1206_3216Metric_Pad1.30x1.75mm_HandSolder"
 			(at 38.862 137.16 90)
 			(effects
@@
 			)
 		)
-		(property "Footprint" ""
+		(property "Footprint" "Capacitor_SMD:C_1206_3216Metric_Pad1.33x1.80mm_HandSolder"
 			(at 51.7652 175.26 0)
 			(effects
@@
 			)
 		)
-		(property "Footprint" ""
+		(property "Footprint" "Diode_SMD:D_SOD-523"
 			(at 182.88 111.76 0)
 			(effects
@@
 			)
 		)
-		(property "Footprint" ""
+		(property "Footprint" "Capacitor_SMD:C_1206_3216Metric_Pad1.33x1.80mm_HandSolder"
 			(at 21.2852 175.26 0)
 			(effects
@@
 			)
 		)
-		(property "Footprint" ""
+		(property "Footprint" "MyFootprints:2x3_ISP_header"
 			(at 201.93 71.12 0)
 			(effects
@@
 			)
 		)
-		(property "Footprint" ""
+		(property "Footprint" "Capacitor_SMD:C_1206_3216Metric_Pad1.33x1.80mm_HandSolder"
 			(at 184.15 49.8348 0)
 			(effects
@@
 			)
 		)
-		(property "Footprint" ""
+		(property "Footprint" "Resistor_SMD:R_1206_3216Metric_Pad1.30x1.75mm_HandSolder"
 			(at 28.702 137.16 90)
 			(effects
@@
 			)
 		)
-		(property "Footprint" ""
+		(property "Footprint" "Capacitor_SMD:C_1206_3216Metric_Pad1.33x1.80mm_HandSolder"
 			(at 31.4452 175.26 0)
 			(effects
@@
 			)
 		)
-		(property "Footprint" ""
+		(property "Footprint" "Capacitor_SMD:C_1206_3216Metric_Pad1.33x1.80mm_HandSolder"
 			(at 184.15 37.1348 0)
 			(effects
@@
 			)
 		)
-		(property "Footprint" ""
+		(property "Footprint" "Package_QFP:TQFP-100_14x14mm_P0.5mm"
 			(at 113.03 104.14 0)
 			(effects
@@
 			)
 		)
-		(property "Footprint" ""
+		(property "Footprint" "Diode_SMD:D_SOD-523"
 			(at 77.47 33.02 0)
 			(effects
@@
 			)
 		)
-		(property "Footprint" ""
+		(property "Footprint" "Capacitor_SMD:C_1206_3216Metric_Pad1.33x1.80mm_HandSolder"
 			(at 53.34 20.6248 0)
 			(effects
