File: KiCad/Open Interface III/Outputs.kicad_sch (KiCad schematic)
At the start: 0 parts

Commit message: OI III Schematics 0.1
Parts:
- added C44, C45, C47, C49: 4.7n, symbol Device:C
- added C46, C48, C50: 100n, symbol Device:C
- added D10, D11, D12, D13, D14, D15, D16, D17, D18, D22, D9: 1N4148, symbol Diode:1N4148
- added D19, D20: Orange, symbol Device:LED
- added D21: Green, symbol Device:LED
- added JP6: REL - ULN, symbol Jumper:Jumper_3_Open
- added K1: G5V-1, symbol Relay:G5V-1
- added R53, R54, R55: 470R, symbol Device:R
- added U17: ULN2803A, symbol Transistor_Array:ULN2803A
Connections:
- new net: D19.2 (A), R53.2
- new net: D10.1 (K), D11.1 (K), D12.1 (K), D9.1 (K), R55.1, U17.7 (I7)
- new net: D21.2 (A), R55.2
- new net: D17.1 (K), D18.1 (K), R53.1
- new net: D13.1 (K), D14.1 (K), R54.1, U17.5 (I5)
- new net: D20.2 (A), R54.2
- new net: D15.1 (K), D16.1 (K), D17.2 (A), U17.1 (I1)
- new net: D22.2 (A), JP6.3 (B), K1.2
- new net: C44.1, JP6.2 (C), U17.12 (O7)
- new net +5V: D22.1 (K), K1.9
- new net CW 232: D15.2 (A)
- new net CW1: D16.2 (A)
- new net CW1 Out: C50.1, U17.18 (O1)
- new net CW2: D18.2 (A), U17.3 (I3)
- new net CW2 Out: C48.1, U17.16 (O3)
- new net FSK: D14.2 (A)
- new net FSK Arduino: D13.2 (A)
- new net FSK Out: C46.1, U17.14 (O5)
- new net GND: C44.2, C45.2, C46.2, C47.2, C48.2, C49.2, C50.2, D19.1 (K), D20.1 (K), D21.1 (K), K1.10, U17.9 (GND)
- new net PA PTT: D12.2 (A)
- new net PA PTT Out: JP6.1 (A), K1.5, K1.6
- new net PTT Mic Out: C45.1, U17.13 (O6)
- new net PTT1: D11.2 (A), U17.2 (I2)
- new net PTT1 Out: C49.1, U17.17 (O2)
- new net PTT2: D10.2 (A), U17.4 (I4)
- new net PTT2 Out: C47.1, U17.15 (O4)
- new net PTT3: D9.2 (A), U17.6 (I6)
- new net SEQ: U17.8 (I8)
- new net SEQ Out: U17.11 (O8)
- new net Vin TRX: U17.10 (COM)
Other:
- note added: "REL - RSY"

Commit message: PCB 0.1, BOM
Parts:
- C44, C45, C46, C47, C48, C49, C50: footprint (none) -> Capacitor_SMD:C_1206_3216Metric_Pad1.33x1.80mm_HandSolder
- D10, D11, D12, D13, D14, D15, D16, D17, D18, D22, D9: footprint (none) -> Diode_SMD:D_SOD-523
- D19, D20, D21: footprint (none) -> MyFootprints:2-pin JST LED
- JP6: footprint (none) -> MyFootprints:Jumper_1x03_P2.54mm_large
- K1: footprint (none) -> Relay_THT:Relay_SPDT_Omron_G5V-1
- R53, R54, R55: footprint (none) -> Resistor_SMD:R_1206_3216Metric_Pad1.30x1.75mm_HandSolder
- U17: footprint (none) -> MyFootprints:DIP-18_W7.62mm w socket
Changed lines of the file:
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@@
 			)
 		)
-		(property "Footprint" ""
+		(property "Footprint" "Capacitor_SMD:C_1206_3216Metric_Pad1.33x1.80mm_HandSolder"
 			(at 197.8152 107.95 0)
 			(effects
@@
 			)
 		)
-		(property "Footprint" ""
+		(property "Footprint" "MyFootprints:2-pin JST LED"
 			(at 87.63 171.45 0)
 			(effects
@@
 			)
 		)
-		(property "Footprint" ""
+		(property "Footprint" "Resistor_SMD:R_1206_3216Metric_Pad1.30x1.75mm_HandSolder"
 			(at 117.602 157.48 90)
 			(effects
@@
 			)
 		)
-		(property "Footprint" ""
+		(property "Footprint" "Resistor_SMD:R_1206_3216Metric_Pad1.30x1.75mm_HandSolder"
 			(at 85.852 157.48 90)
 			(effects
@@
 			)
 		)
-		(property "Footprint" ""
+		(property "Footprint" "Diode_SMD:D_SOD-523"
 			(at 52.07 78.74 0)
 			(effects
@@
 			)
 		)
-		(property "Footprint" ""
+		(property "Footprint" "Resistor_SMD:R_1206_3216Metric_Pad1.30x1.75mm_HandSolder"
 			(at 102.362 157.48 90)
 			(effects
@@
 			)
 		)
-		(property "Footprint" ""
+		(property "Footprint" "Diode_SMD:D_SOD-523"
 			(at 52.07 64.77 0)
 			(effects
@@
 			)
 		)
-		(property "Footprint" ""
+		(property "Footprint" "Diode_SMD:D_SOD-523"
 			(at 71.12 138.43 0)
 			(effects
@@
 			)
 		)
-		(property "Footprint" ""
+		(property "Footprint" "Capacitor_SMD:C_1206_3216Metric_Pad1.33x1.80mm_HandSolder"
 			(at 235.9152 107.95 0)
 			(effects
@@
 			)
 		)
-		(property "Footprint" ""
+		(property "Footprint" "Capacitor_SMD:C_1206_3216Metric_Pad1.33x1.80mm_HandSolder"
 			(at 185.1152 107.95 0)
 			(effects
@@
 			)
 		)
-		(property "Footprint" ""
+		(property "Footprint" "Diode_SMD:D_SOD-523"
 			(at 207.01 43.18 0)
 			(effects
@@
 			)
 		)
-		(property "Footprint" ""
+		(property "Footprint" "Diode_SMD:D_SOD-523"
 			(at 52.07 106.68 0)
 			(effects
@@
 			)
 		)
-		(property "Footprint" ""
+		(property "Footprint" "Diode_SMD:D_SOD-523"
 			(at 52.07 48.26 0)
 			(effects
@@
 			)
 		)
-		(property "Footprint" ""
+		(property "Footprint" "Diode_SMD:D_SOD-523"
 			(at 52.07 92.71 0)
 			(effects
@@
 			)
 		)
-		(property "Footprint" ""
+		(property "Footprint" "Capacitor_SMD:C_1206_3216Metric_Pad1.33x1.80mm_HandSolder"
 			(at 223.2152 107.95 0)
 			(effects
@@
 			)
 		)
-		(property "Footprint" ""
+		(property "Footprint" "MyFootprints:Jumper_1x03_P2.54mm_large"
 			(at 184.15 44.45 0)
 			(effects
@@
 			)
 		)
-		(property "Footprint" ""
+		(property "Footprint" "MyFootprints:2-pin JST LED"
 			(at 119.38 171.45 0)
 			(effects
@@
 			)
 		)
-		(property "Footprint" ""
+		(property "Footprint" "Diode_SMD:D_SOD-523"
 			(at 52.07 36.83 0)
 			(effects
@@
 			)
 		)
-		(property "Footprint" ""
+		(property "Footprint" "Capacitor_SMD:C_1206_3216Metric_Pad1.33x1.80mm_HandSolder"
 			(at 172.4152 107.95 0)
 			(effects
@@
 			)
 		)
-		(property "Footprint" ""
+		(property "Footprint" "Diode_SMD:D_SOD-523"
 			(at 52.07 25.4 0)
 			(effects
@@
 			)
 		)
-		(property "Footprint" ""
+		(property "Footprint" "Capacitor_SMD:C_1206_3216Metric_Pad1.33x1.80mm_HandSolder"
 			(at 210.5152 107.95 0)
 			(effects
@@
 			)
 		)
-		(property "Footprint" ""
+		(property "Footprint" "Relay_THT:Relay_SPDT_Omron_G5V-1"
 			(at 264.922 42.418 0)
 			(effects
@@
 			)
 		)
-		(property "Footprint" ""
+		(property "Footprint" "Capacitor_SMD:C_1206_3216Metric_Pad1.33x1.80mm_HandSolder"
 			(at 248.6152 107.95 0)
 			(effects
@@
 			)
 		)
-		(property "Footprint" ""
+		(property "Footprint" "Diode_SMD:D_SOD-523"
 			(at 52.07 119.38 0)
 			(effects
@@
 			)
 		)
-		(property "Footprint" ""
+		(property "Footprint" "MyFootprints:2-pin JST LED"
 			(at 104.14 171.45 0)
 			(effects
@@
 			)
 		)
-		(property "Footprint" ""
+		(property "Footprint" "Diode_SMD:D_SOD-523"
 			(at 87.63 138.43 0)
 			(effects
@@
 			)
 		)
-		(property "Footprint" ""
+		(property "Footprint" "MyFootprints:DIP-18_W7.62mm w socket"
 			(at 157.48 90.17 0)
 			(effects
