File: KiCad/Open Interface III/TRX_CAT.kicad_sch (KiCad schematic)
At the start: 0 parts

Commit message: OI III Schematics 0.1
Parts:
- added C51, C55, C56, C57, C58: 1u, symbol Device:C_Polarized
- added C52: 100n, symbol Device:C
- added C53, C54: 22p, symbol Device:C
- added D23, D24: Green, symbol Device:LED
- added D25, D30: 1N4148, symbol Diode:1N4148
- added D26, D27, D28, D29: D_Zener, symbol Device:D_Zener
- added J8: Conn_02x04_Odd_Even, symbol Connector_Generic:Conn_02x04_Odd_Even
- added L26: L, symbol Device:L
- added R56: 1k5, symbol Device:R
- added R57, R58: 15k, symbol Device:R
- added R59, R60: 27R, symbol Device:R
- added R61, R62: 470R, symbol Device:R
- added R63: 4k7, symbol Device:R
- added R64: 1k, symbol Device:R
- added R65, R66: 220R, symbol Device:R
- added U18: FT232RL, symbol Interface_USB:FT232RL
- added U19: MAX232, symbol Interface_UART:MAX232
Connections:
- new net: C58.2, U19.6 (VS-)
- new net: D25.1 (K), U18.1 (TXD)
- new net: D25.2 (A), D30.2 (A), J8.4 (Pin_4), R63.2
- new net: R56.2, R57.1, R59.1, U18.15 (USBD+)
- new net: R58.1, R60.1, U18.16 (USBD-)
- new net: C51.2, L26.2, U18.20 (VCC), U18.4 (VCCIO)
- new net: R61.1, U18.22 (CBUS1)
- new net: D23.2 (A), R61.2
- new net: J8.1 (Pin_1), U19.14 (T1OUT)
- new net: J8.2 (Pin_2), U19.11 (T1IN)
- new net: J8.3 (Pin_3), R65.2
- new net: J8.5 (Pin_5), U19.13 (R1IN)
- new net: J8.6 (Pin_6), U19.12 (R1OUT)
- new net: J8.7 (Pin_7), R66.2
- new net: J8.8 (Pin_8), R64.2, U18.5 (RXD)
- new net: D28.2 (A), D29.2 (A)
- new net: D26.2 (A), D27.2 (A)
- new net: C56.1, U19.4 (C2+)
- new net: C56.2, U19.5 (C2-)
- new net: C52.1, U18.17 (3V3OUT)
- new net: R62.1, U18.23 (CBUS0)
- new net: C55.1, U19.1 (C1+)
- new net: C57.2, U19.2 (VS+)
- new net: C55.2, U19.3 (C1-)
- new net: D24.2 (A), R62.2
- new net +3.3V: R56.1
- new net +5V: C57.1, D23.1 (K), D24.1 (K), L26.1, R63.1, U19.16 (VCC)
- new net CAT RxD: R65.1
- new net CAT TxD: D28.1 (K), R66.1
- new net GND: C51.1, C52.2, C53.2, C54.2, C58.1, D27.1 (K), D29.1 (K), R57.2, R58.2, U18.18 (GND), U18.21 (GND), U18.25 (AGND), U18.26 (TEST), U18.7 (GND), U19.15 (GND)
- new net Reset: U18.19 (~{RESET})
- new net RxD2: R64.1
- new net TxD2: D30.1 (K)
- new net USB2+: C53.1, R59.2
- new net USB2-: C54.1, R60.2

Commit message: PCB 0.1, BOM
Parts:
- C51, C55, C56, C57, C58: footprint (none) -> Capacitor_SMD:CP_Elec_5x5.4
- C52, C53, C54: footprint (none) -> Capacitor_SMD:C_1206_3216Metric_Pad1.33x1.80mm_HandSolder
- D23, D24: footprint (none) -> MyFootprints:2-pin JST LED
- D25, D30: footprint (none) -> Diode_SMD:D_SOD-523
- D26, D27, D28, D29: footprint (none) -> Package_TO_SOT_SMD:SOT-23_Handsoldering
- J8: footprint (none) -> Connector_PinHeader_2.54mm:PinHeader_2x04_P2.54mm_Vertical
- L26: footprint (none) -> Inductor_SMD:L_1206_3216Metric_Pad1.22x1.90mm_HandSolder
- R56, R57, R58, R59, R60, R61, R62, R63, R64, R65, R66: footprint (none) -> Resistor_SMD:R_1206_3216Metric_Pad1.30x1.75mm_HandSolder
- U18: footprint (none) -> Package_SO:SSOP-28_5.3x10.2mm_P0.65mm
- U19: footprint (none) -> Package_SO:SOIC-16_3.9x9.9mm_P1.27mm
Connections:
- net CAT RxD: now also D26.1 (K)
Changed lines of the file:
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@@
 	(wire
 		(pts
+			(xy 148.59 144.78) (xy 148.59 162.56)
+		)
+		(stroke
+			(width 0)
+			(type default)
+		)
+	)
+	(wire
+		(pts
 			(xy 133.35 40.64) (xy 133.35 45.72)
 		)
@@
 	(wire
 		(pts
-			(xy 148.59 144.78) (xy 148.59 161.29)
-		)
-		(stroke
-			(width 0)
-			(type default)
-		)
-	)
-	(wire
-		(pts
 			(xy 148.59 182.88) (xy 148.59 187.96)
 		)
@@
 			)
 		)
-		(property "Footprint" ""
+		(property "Footprint" "Capacitor_SMD:CP_Elec_5x5.4"
 			(at 265.1252 85.09 0)
 			(effects
@@
 			)
 		)
-		(property "Footprint" ""
+		(property "Footprint" "Diode_SMD:D_SOD-523"
 			(at 124.46 58.42 0)
 			(effects
@@
 			)
 		)
-		(property "Footprint" ""
+		(property "Footprint" "Diode_SMD:D_SOD-523"
 			(at 168.91 106.68 0)
 			(effects
@@
 			)
 		)
-		(property "Footprint" ""
+		(property "Footprint" "Resistor_SMD:R_1206_3216Metric_Pad1.30x1.75mm_HandSolder"
 			(at 74.93 24.638 90)
 			(effects
@@
 			)
 		)
-		(property "Footprint" ""
+		(property "Footprint" "Resistor_SMD:R_1206_3216Metric_Pad1.30x1.75mm_HandSolder"
 			(at 74.93 34.798 90)
 			(effects
@@
 			)
 		)
-		(property "Footprint" ""
+		(property "Footprint" "Capacitor_SMD:CP_Elec_5x5.4"
 			(at 18.0848 107.95 0)
 			(effects
@@
 			)
 		)
-		(property "Footprint" ""
+		(property "Footprint" "Capacitor_SMD:C_1206_3216Metric_Pad1.33x1.80mm_HandSolder"
 			(at 160.9852 53.34 0)
 			(effects
@@
 			)
 		)
-		(property "Footprint" ""
+		(property "Footprint" "Resistor_SMD:R_1206_3216Metric_Pad1.30x1.75mm_HandSolder"
 			(at 101.6 127.508 90)
 			(effects
@@
 			)
 		)
-		(property "Footprint" ""
+		(property "Footprint" "Connector_PinHeader_2.54mm:PinHeader_2x04_P2.54mm_Vertical"
 			(at 190.5 109.22 0)
 			(effects
@@
 			)
 		)
-		(property "Footprint" ""
+		(property "Footprint" "Package_TO_SOT_SMD:SOT-23_Handsoldering"
 			(at 162.56 166.37 0)
 			(effects
@@
 			)
 		)
-		(property "Footprint" ""
+		(property "Footprint" "Package_TO_SOT_SMD:SOT-23_Handsoldering"
 			(at 148.59 166.37 0)
 			(effects
@@
 			)
 		)
-		(property "Footprint" ""
+		(property "Footprint" "Resistor_SMD:R_1206_3216Metric_Pad1.30x1.75mm_HandSolder"
 			(at 168.91 93.218 90)
 			(effects
@@
 			)
 		)
-		(property "Footprint" ""
+		(property "Footprint" "Capacitor_SMD:CP_Elec_5x5.4"
 			(at 252.73 38.4048 0)
 			(effects
@@
 			)
 		)
-		(property "Footprint" ""
+		(property "Footprint" "Package_TO_SOT_SMD:SOT-23_Handsoldering"
 			(at 162.56 179.07 0)
 			(effects
@@
 			)
 		)
-		(property "Footprint" ""
+		(property "Footprint" "Package_SO:SSOP-28_5.3x10.2mm_P0.65mm"
 			(at 123.19 99.06 0)
 			(effects
@@
 			)
 		)
-		(property "Footprint" ""
+		(property "Footprint" "Package_SO:SOIC-16_3.9x9.9mm_P1.27mm"
 			(at 220.98 88.9 0)
 			(effects
@@
 			)
 		)
-		(property "Footprint" ""
+		(property "Footprint" "MyFootprints:2-pin JST LED"
 			(at 88.9 125.73 0)
 			(effects
@@
 			)
 		)
-		(property "Footprint" ""
+		(property "Footprint" "Capacitor_SMD:C_1206_3216Metric_Pad1.33x1.80mm_HandSolder"
 			(at 150.8252 45.72 0)
 			(effects
@@
 			)
 		)
-		(property "Footprint" ""
+		(property "Footprint" "Resistor_SMD:R_1206_3216Metric_Pad1.30x1.75mm_HandSolder"
 			(at 176.53 146.558 90)
 			(effects
@@
 			)
 		)
-		(property "Footprint" ""
+		(property "Footprint" "Resistor_SMD:R_1206_3216Metric_Pad1.30x1.75mm_HandSolder"
 			(at 131.572 49.53 90)
 			(effects
@@
 			)
 		)
-		(property "Footprint" ""
+		(property "Footprint" "Inductor_SMD:L_1206_3216Metric_Pad1.22x1.90mm_HandSolder"
 			(at 19.05 31.75 0)
 			(effects
@@
 			)
 		)
-		(property "Footprint" ""
+		(property "Footprint" "Resistor_SMD:R_1206_3216Metric_Pad1.30x1.75mm_HandSolder"
 			(at 42.672 113.03 90)
 			(effects
@@
 			)
 		)
-		(property "Footprint" ""
+		(property "Footprint" "Package_TO_SOT_SMD:SOT-23_Handsoldering"
 			(at 148.59 179.07 0)
 			(effects
@@
 			)
 		)
-		(property "Footprint" ""
+		(property "Footprint" "Resistor_SMD:R_1206_3216Metric_Pad1.30x1.75mm_HandSolder"
 			(at 176.53 159.258 90)
 			(effects
@@
 			)
 		)
-		(property "Footprint" ""
+		(property "Footprint" "MyFootprints:2-pin JST LED"
 			(at 88.9 138.43 0)
 			(effects
@@
 			)
 		)
-		(property "Footprint" ""
+		(property "Footprint" "Resistor_SMD:R_1206_3216Metric_Pad1.30x1.75mm_HandSolder"
 			(at 52.832 113.03 90)
 			(effects
@@
 			)
 		)
-		(property "Footprint" ""
+		(property "Footprint" "Resistor_SMD:R_1206_3216Metric_Pad1.30x1.75mm_HandSolder"
 			(at 42.672 30.48 90)
 			(effects
@@
 			)
 		)
-		(property "Footprint" ""
+		(property "Footprint" "Resistor_SMD:R_1206_3216Metric_Pad1.30x1.75mm_HandSolder"
 			(at 101.6 140.208 90)
 			(effects
@@
 			)
 		)
-		(property "Footprint" ""
+		(property "Footprint" "Capacitor_SMD:CP_Elec_5x5.4"
 			(at 186.69 38.4048 0)
 			(effects
@@
 			)
 		)
-		(property "Footprint" ""
+		(property "Footprint" "Capacitor_SMD:C_1206_3216Metric_Pad1.33x1.80mm_HandSolder"
 			(at 32.7152 116.84 0)
 			(effects
@@
 			)
 		)
-		(property "Footprint" ""
+		(property "Footprint" "Capacitor_SMD:CP_Elec_5x5.4"
 			(at 263.1948 43.18 0)
 			(effects
