File: KiCad/Open Interface III/USB Sound Card.kicad_sch (KiCad schematic)
At the start: 0 parts

Commit message: OI III Schematics 0.1
Parts:
- added C59, C65, C66, C77, C79: 10u, symbol Device:C_Polarized
- added C60, C61, C78, C80: 22p, symbol Device:C
- added C62: 10, symbol Device:C_Polarized
- added C63: 100n, symbol Device:C
- added C64: 47u, symbol Device:C_Polarized
- added C67, C71, C72, C75, C81, C82: 1u, symbol Device:C_Polarized
- added C68, C74: 1n, symbol Device:C
- added C69, C73: 10u, symbol Device:C
- added C70: 68n, symbol Device:C
- added C76: 4.7u, symbol Device:C_Polarized
- added D31, D32, D33, D34: 1N4148, symbol Diode:1N4148
- added L27: L, symbol Device:L
- added Q4: BC817, symbol Transistor_BJT:BC817
- added R67, R71: 27R, symbol Device:R
- added R68, R76, R77, R78, R82: 4k7, symbol Device:R
- added R69, R75: 100k, symbol Device:R
- added R70, R79: 470R, symbol Device:R
- added R72, R74: 15k, symbol Device:R
- added R73: 1k5, symbol Device:R
- added R80: 1k, symbol Device:R
- added R81: 1M, symbol Device:R
- added RV4: 10k log, symbol Device:R_Potentiometer
- added T1, T2: Transformer_1P_1S_SO8, symbol Device:Transformer_1P_1S_SO8
- added U20: Vol -, symbol My_Parts:Switch
- added U21: Vol +, symbol My_Parts:Switch
- added U22: Mute, symbol My_Parts:Switch
- added U23: PCM2904, symbol My_Parts:PCM2904
- added Y3: Crystal, symbol Device:Crystal
Connections:
- new net: C82.1, L27.2, U23.3 (VBUS)
- new net: R67.2, R72.2, U23.2 (D-)
- new net: R71.2, R73.2, R74.2, U23.1 (D+)
- new net: C77.1, U23.10 (VCCCI)
- new net: C65.1, U23.12 (VINL)
- new net: C62.1, U23.13 (VINR)
- new net: C76.1, U23.14 (VCOM)
- new net: C81.1, U23.15 (VOUTR)
- new net: C79.1, U23.16 (VOUTL)
- new net: C75.1, U23.17 (VCCP1I)
- new net: C72.1, U23.19 (VCCP2I)
- new net: C78.1, R81.1, U23.20 (XTO), Y3.1
- new net: C80.1, R81.2, U23.21 (XTI), Y3.2
- new net: C71.1, U23.23 (VCCXI)
- new net: C67.1, U23.27 (VDDI), U23.8 (SEL0), U23.9 (SEL1)
- new net: R76.1, R77.1, R78.1, U23.28 (~{SSPND})
- new net: U22.2 (NO), U23.5 (HID0)
- new net: U21.2 (NO), U23.6 (HID1)
- new net: U20.2 (NO), U23.7 (HID2)
- new net: R77.2, U21.1 (Com)
- new net: C66.1, Q4.1 (B), R69.2, R75.1
- new net: C66.2, RV4.2
- new net: D33.2 (A), D34.1 (K)
- new net: C73.2, T2.1 (AA)
- new net: C74.2, T2.4 (AB)
- new net: R80.1, R82.1, T2.8 (SB)
- new net: RV4.1, T1.8 (SB)
- new net: RV4.3, T1.5 (SA)
- new net: C69.2, T1.1 (AA)
- new net: C59.1, Q4.3 (C), R68.1, R69.1
- new net: C59.2, C62.2, C65.2, D31.2 (A), D33.1 (K)
- new net: C73.1, R79.2
- new net: C79.2, C81.2, R82.2
- new net: D31.1 (K), D32.2 (A)
- new net: C64.1, Q4.2 (E), R70.1
- new net: R76.2, U20.1 (Com)
- new net: R78.2, U22.1 (Com)
- new net: C63.1, R68.2
- new net +3.3V: R73.1
- new net +5V: L27.1
- new net AGNDC: C64.2, D32.1 (K), D34.2 (A), R70.2, R75.2, U23.11 (AGNDC)
- new net GND: C60.2, C61.2, C63.2, C67.2, C71.2, C72.2, C75.2, C76.2, C77.2, C78.2, C80.2, C82.2, R72.1, R74.1, U23.18 (AGNDP), U23.22 (AGNDX), U23.24 (TEST0), U23.26 (DGND), U23.4 (DGNDU)
- new net Rx Audio: C68.1, C69.1
- new net Rx Audio GND: C68.2, T1.4 (AB)
- new net Tx Audio GND: C70.2, C74.1
- new net Tx Sound: C70.1, R79.1
- new net USB3+: C61.1, R71.1
- new net USB3-: C60.1, R67.1
- new net VGNDC: R80.2, T2.5 (SA)

Commit message: PCB 0.1, BOM
Parts:
- removed T1, T2: Transformer_1P_1S_SO8, symbol Device:Transformer_1P_1S_SO8
- added T1, T2: Transformer_1P_1S, MyFootprints:Audio Transformer Bourns SM-LP-5001, symbol Device:Transformer_1P_1S
- C59, C65, C66, C67, C71, C72, C75, C77, C79, C81, C82: footprint (none) -> Capacitor_SMD:CP_Elec_5x5.4
- C60, C61, C63, C68, C69, C70, C73, C74, C78, C80: footprint (none) -> Capacitor_SMD:C_1206_3216Metric_Pad1.33x1.80mm_HandSolder
- C62: value 10 -> 10u; footprint (none) -> Capacitor_SMD:CP_Elec_5x5.4
- C64: footprint (none) -> Capacitor_SMD:CP_Elec_6.3x5.8
- C76: footprint (none) -> Capacitor_SMD:CP_Elec_4x5.4
- D31, D32, D33, D34: footprint (none) -> Diode_SMD:D_SOD-523
- L27: footprint (none) -> Inductor_SMD:L_1206_3216Metric_Pad1.22x1.90mm_HandSolder
- Q4: footprint (none) -> Package_TO_SOT_SMD:SOT-23-3
- R67, R68, R69, R70, R71, R72, R73, R74, R75, R76, R77, R78, R79, R80, R81, R82: footprint (none) -> Resistor_SMD:R_1206_3216Metric_Pad1.30x1.75mm_HandSolder
- RV4: footprint (none) -> MyFootprints:3-pin JST Potentiometer
- U20, U21, U22: footprint (none) -> MyFootprints:2-pin JST Switch
- U23: footprint (none) -> Package_SO:SSOP-28_5.3x10.2mm_P0.65mm
- Y3: value Crystal -> 12 MHz; footprint (none) -> Crystal:Crystal_SMD_HC49-SD
Connections:
- net Rx Audio GND: now also T1.3 (SA)
- net VGNDC: now also T2.3 (SA)
- net at C73.2: now also T2.1 (AA)
- net at C74.2: now also T2.2 (AB)
- net at R80.1, R82.1: now also T2.4 (SB)
- net at RV4.1: now also T1.1 (AA)
- net at RV4.3: now also T1.2 (AB)
- net at C69.2: now also T1.4 (SB)
