File: KiCad/Open Interface III/USB_Hub.kicad_sch (KiCad schematic)
At the start: 11 parts, among them U3 TUSB2046B, Y1 6MHz

Commit message: OI III Schematics 0.1
Parts:
- U5: renamed from U3; footprint Package_QFP:LQFP-32_7x7mm_P0.8mm -> (none)
- renumbered C6 to C17, C5 to C18, C7 to C19, C8 to C20, R6 to R14, R5 to R15, R4 to R16, R8 to R17, R7 to R18, Y1 to Y2
Changed lines of the file:
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@@
 	(generator_version "8.0")
 	(paper "A4")
+	(title_block
+		(rev "0.1")
+	)
 	(junction
 		(at 81.28 133.35)
@@
 		(dnp no)
 		(fields_autoplaced yes)
-		(property "Reference" "Y1"
+		(property "Reference" "Y2"
 			(at 120.65 149.86 0)
 			(effects
@@
 			(project ""
 				(path "/d93537ee-5c24-4c3e-8ba0-9c6559a17368/984810fb-07e9-4dc7-899a-8d7391d09c8c"
-					(reference "Y1")
+					(reference "Y2")
 					(unit 1)
 				)
@@
 		(dnp no)
 		(fields_autoplaced yes)
-		(property "Reference" "#PWR5"
+		(property "Reference" "#PWR17"
 			(at 172.72 144.78 0)
 			(effects
@@
 			(project ""
 				(path "/d93537ee-5c24-4c3e-8ba0-9c6559a17368/984810fb-07e9-4dc7-899a-8d7391d09c8c"
-					(reference "#PWR5")
+					(reference "#PWR17")
 					(unit 1)
 				)
@@
 		(dnp no)
 		(fields_autoplaced yes)
-		(property "Reference" "C7"
+		(property "Reference" "C19"
 			(at 113.03 167.6399 0)
 			(effects
@@
 			(project ""
 				(path "/d93537ee-5c24-4c3e-8ba0-9c6559a17368/984810fb-07e9-4dc7-899a-8d7391d09c8c"
-					(reference "C7")
+					(reference "C19")
 					(unit 1)
 				)
@@
 		(dnp no)
 		(fields_autoplaced yes)
-		(property "Reference" "U3"
+		(property "Reference" "U5"
 			(at 179.9941 46.99 0)
 			(effects
@@
 			)
 		)
-		(property "Footprint" "Package_QFP:LQFP-32_7x7mm_P0.8mm"
+		(property "Footprint" ""
 			(at 201.93 125.73 0)
 			(effects
@@
 			(project ""
 				(path "/d93537ee-5c24-4c3e-8ba0-9c6559a17368/984810fb-07e9-4dc7-899a-8d7391d09c8c"
-					(reference "U3")
+					(reference "U5")
 					(unit 1)
 				)
@@
 		(dnp no)
 		(fields_autoplaced yes)
-		(property "Reference" "R4"
+		(property "Reference" "R16"
 			(at 95.25 82.5499 0)
 			(effects
@@
 			(project ""
 				(path "/d93537ee-5c24-4c3e-8ba0-9c6559a17368/984810fb-07e9-4dc7-899a-8d7391d09c8c"
-					(reference "R4")
+					(reference "R16")
 					(unit 1)
 				)
@@
 		(dnp no)
 		(fields_autoplaced yes)
-		(property "Reference" "R7"
+		(property "Reference" "R18"
 			(at 120.65 137.16 90)
 			(effects
@@
 			(project ""
 				(path "/d93537ee-5c24-4c3e-8ba0-9c6559a17368/984810fb-07e9-4dc7-899a-8d7391d09c8c"
-					(reference "R7")
+					(reference "R18")
 					(unit 1)
 				)
@@
 		(dnp no)
 		(fields_autoplaced yes)
-		(property "Reference" "#PWR4"
+		(property "Reference" "#PWR18"
 			(at 210.82 30.48 0)
 			(effects
@@
 			(project ""
 				(path "/d93537ee-5c24-4c3e-8ba0-9c6559a17368/984810fb-07e9-4dc7-899a-8d7391d09c8c"
-					(reference "#PWR4")
+					(reference "#PWR18")
 					(unit 1)
 				)
@@
 		(dnp no)
 		(fields_autoplaced yes)
-		(property "Reference" "R5"
+		(property "Reference" "R15"
 			(at 83.82 55.8799 0)
 			(effects
@@
 			(project "Open Interface III"
 				(path "/d93537ee-5c24-4c3e-8ba0-9c6559a17368/984810fb-07e9-4dc7-899a-8d7391d09c8c"
-					(reference "R5")
+					(reference "R15")
 					(unit 1)
 				)
@@
 		(dnp no)
 		(fields_autoplaced yes)
-		(property "Reference" "C8"
+		(property "Reference" "C20"
 			(at 135.89 167.6399 0)
 			(effects
@@
 			(project "Open Interface III"
 				(path "/d93537ee-5c24-4c3e-8ba0-9c6559a17368/984810fb-07e9-4dc7-899a-8d7391d09c8c"
-					(reference "C8")
+					(reference "C20")
 					(unit 1)
 				)
@@
 		(dnp no)
 		(fields_autoplaced yes)
-		(property "Reference" "C6"
+		(property "Reference" "C17"
 			(at 72.39 82.5499 0)
 			(effects
@@
 			(project "Open Interface III"
 				(path "/d93537ee-5c24-4c3e-8ba0-9c6559a17368/984810fb-07e9-4dc7-899a-8d7391d09c8c"
-					(reference "C6")
+					(reference "C17")
 					(unit 1)
 				)
@@
 		(dnp no)
 		(fields_autoplaced yes)
-		(property "Reference" "C5"
+		(property "Reference" "C18"
 			(at 85.09 82.5499 0)
 			(effects
@@
 			(project ""
 				(path "/d93537ee-5c24-4c3e-8ba0-9c6559a17368/984810fb-07e9-4dc7-899a-8d7391d09c8c"
-					(reference "C5")
+					(reference "C18")
 					(unit 1)
 				)
@@
 		(dnp no)
 		(fields_autoplaced yes)
-		(property "Reference" "#PWR6"
+		(property "Reference" "#PWR16"
 			(at 109.22 191.77 0)
 			(effects
@@
 			(project ""
 				(path "/d93537ee-5c24-4c3e-8ba0-9c6559a17368/984810fb-07e9-4dc7-899a-8d7391d09c8c"
-					(reference "#PWR6")
+					(reference "#PWR16")
 					(unit 1)
 				)
@@
 		(dnp no)
 		(fields_autoplaced yes)
-		(property "Reference" "R6"
+		(property "Reference" "R14"
 			(at 71.12 55.8799 0)
 			(effects
@@
 			(project "Open Interface III"
 				(path "/d93537ee-5c24-4c3e-8ba0-9c6559a17368/984810fb-07e9-4dc7-899a-8d7391d09c8c"
-					(reference "R6")
+					(reference "R14")
 					(unit 1)
 				)
@@
 		(dnp no)
 		(fields_autoplaced yes)
-		(property "Reference" "R8"
+		(property "Reference" "R17"
 			(at 119.38 111.76 90)
 			(effects
@@
 			(project ""
 				(path "/d93537ee-5c24-4c3e-8ba0-9c6559a17368/984810fb-07e9-4dc7-899a-8d7391d09c8c"
-					(reference "R8")
+					(reference "R17")
 					(unit 1)
 				)

Commit message: PCB 0.1, BOM
Parts:
- C17, C18, C19, C20: footprint (none) -> Capacitor_SMD:C_1206_3216Metric_Pad1.33x1.80mm_HandSolder
- R14, R15, R16, R17, R18: footprint (none) -> Resistor_SMD:R_1206_3216Metric_Pad1.30x1.75mm_HandSolder
- U5: footprint (none) -> Package_QFP:LQFP-32_7x7mm_P0.8mm
- Y2: footprint (none) -> Crystal:Crystal_SMD_HC49-SD
Changed lines of the file:
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@@
 			)
 		)
-		(property "Footprint" ""
+		(property "Footprint" "Crystal:Crystal_SMD_HC49-SD"
 			(at 120.65 157.48 0)
 			(effects
@@
 			)
 		)
-		(property "Footprint" ""
+		(property "Footprint" "Capacitor_SMD:C_1206_3216Metric_Pad1.33x1.80mm_HandSolder"
 			(at 110.1852 172.72 0)
 			(effects
@@
 			)
 		)
-		(property "Footprint" ""
+		(property "Footprint" "Package_QFP:LQFP-32_7x7mm_P0.8mm"
 			(at 201.93 125.73 0)
 			(effects
@@
 			)
 		)
-		(property "Footprint" ""
+		(property "Footprint" "Resistor_SMD:R_1206_3216Metric_Pad1.30x1.75mm_HandSolder"
 			(at 90.932 83.82 90)
 			(effects
@@
 			)
 		)
-		(property "Footprint" ""
+		(property "Footprint" "Resistor_SMD:R_1206_3216Metric_Pad1.30x1.75mm_HandSolder"
 			(at 120.65 145.288 90)
 			(effects
@@
 			)
 		)
-		(property "Footprint" ""
+		(property "Footprint" "Resistor_SMD:R_1206_3216Metric_Pad1.30x1.75mm_HandSolder"
 			(at 79.502 57.15 90)
 			(effects
@@
 			)
 		)
-		(property "Footprint" ""
+		(property "Footprint" "Capacitor_SMD:C_1206_3216Metric_Pad1.33x1.80mm_HandSolder"
 			(at 133.0452 172.72 0)
 			(effects
@@
 			)
 		)
-		(property "Footprint" ""
+		(property "Footprint" "Capacitor_SMD:C_1206_3216Metric_Pad1.33x1.80mm_HandSolder"
 			(at 69.5452 87.63 0)
 			(effects
@@
 			)
 		)
-		(property "Footprint" ""
+		(property "Footprint" "Capacitor_SMD:C_1206_3216Metric_Pad1.33x1.80mm_HandSolder"
 			(at 82.2452 87.63 0)
 			(effects
@@
 			)
 		)
-		(property "Footprint" ""
+		(property "Footprint" "Resistor_SMD:R_1206_3216Metric_Pad1.30x1.75mm_HandSolder"
 			(at 66.802 57.15 90)
 			(effects
@@
 			)
 		)
-		(property "Footprint" ""
+		(property "Footprint" "Resistor_SMD:R_1206_3216Metric_Pad1.30x1.75mm_HandSolder"
 			(at 119.38 119.888 90)
 			(effects
